File: radar.sch (KiCad schematic (older format))
At the start: 13 parts, among them J102 Conn_01x01, J103 Conn_01x01, J105 Conn_01x01, J106 Conn_01x02, J108 Conn_Coaxial, J109 Conn_Coaxial

Commit message: Switch signal conditioning to fully differential
Parts:
- removed J105: Conn_01x01, Connectors:1pin, symbol Conn_01x01
- added J?: Conn_01x02, symbol Conn_01x02
Connections:
- new net BASEBAND/OUT+: J?.1 (Pin_1)
- new net BASEBAND/OUT-: J?.2 (Pin_2)
Other:
- moved on the sheet: J106, J109
Changed lines of the file:
@@
 $EndSheet
 $Sheet
-S 3320 2785 2090 1190
+S 4485 2785 1505 1180
 U 59D58014
 F0 "INPUT_AMP" 60
 F1 "input.sch" 60
-F2 "RF_IN" I L 3320 3385 60
-F3 "RF_OUT" I R 5410 3305 60
-F4 "EN1" I L 3320 3665 60
-F5 "EN2" I L 3320 3765 60
+F2 "RF_IN" I L 4485 3385 60
+F3 "RF_OUT" I R 5990 3305 60
+F4 "EN1" I L 4485 3665 60
+F5 "EN2" I L 4485 3765 60
 $EndSheet
 $Sheet
@@
 F2 "INP" I L 9030 2875 60
 F3 "INM" I L 9030 2985 60
-F4 "OUT" I R 10210 2925 60
+F4 "OUT+" I R 10210 2870 60
+F5 "OUT-" I R 10210 2970 60
 $EndSheet
 Text Notes 7915 3805 0    60   ~ 0
 +0 dB, 5V 60mA
-Text Notes 3710 4155 0    60   ~ 0
+Text Notes 4875 4155 0    60   ~ 0
 +0-30 dB, 3.3V 30mA
 Text Notes 9260 3825 0    60   ~ 0
 12 V, 10mA
 Wire Wire Line
-	5410 3305 7795 3305
-Wire Wire Line
-	1770 2755 3040 2755
+	2935 2755 4205 2755
 Wire Wire Line
 	2915 1650 3955 1650
 $Sheet
-S 1450 3325 1380 690
+S 2615 3325 1380 690
 U 5A51736E
 F0 "LEVELSHIFTER" 60
 F1 "levelshifter.sch" 60
-F2 "OUT1" I R 2830 3665 60
-F3 "OUT2" I R 2830 3765 60
-F4 "IN1" I L 1450 3665 60
-F5 "IN2" I L 1450 3765 60
-$EndSheet
-Wire Wire Line
-	3040 2755 3040 3385
-Wire Wire Line
-	3040 3385 3320 3385
-Wire Wire Line
-	2830 3665 3320 3665
-Wire Wire Line
-	2830 3765 3320 3765
+F2 "OUT1" I R 3995 3665 60
+F3 "OUT2" I R 3995 3765 60
+F4 "IN1" I L 2615 3665 60
+F5 "IN2" I L 2615 3765 60
+$EndSheet
+Wire Wire Line
+	4205 2755 4205 3385
+Wire Wire Line
+	4205 3385 4485 3385
+Wire Wire Line
+	3995 3665 4485 3665
+Wire Wire Line
+	3995 3765 4485 3765
 $Comp
 L Conn_01x02 J106
 U 1 1 5A51B599
-P 1040 3665
-F 0 "J106" H 1040 3765 50  0000 C CNN
-F 1 "Conn_01x02" H 1040 3465 50  0000 C CNN
-F 2 "Socket_Strips:Socket_Strip_Straight_1x02_Pitch2.54mm" H 1040 3665 50  0001 C CNN
-F 3 "" H 1040 3665 50  0001 C CNN
-	1    1040 3665
-	-1   0    0    -1
-$EndComp
-Wire Wire Line
-	1240 3665 1450 3665
-Wire Wire Line
-	1240 3765 1450 3765
+P 2205 3665
+F 0 "J106" H 2205 3765 50  0000 C CNN
+F 1 "Conn_01x02" H 2205 3465 50  0000 C CNN
+F 2 "Socket_Strips:Socket_Strip_Straight_1x02_Pitch2.54mm" H 2205 3665 50  0001 C CNN
+F 3 "" H 2205 3665 50  0001 C CNN
+	1    2205 3665
+	-1   0    0    -1
+$EndComp
+Wire Wire Line
+	2405 3665 2615 3665
+Wire Wire Line
+	2405 3765 2615 3765
 $Comp
 L Conn_01x01 J103
@@
 	5235 1810 5085 1810
 $Comp
-L Conn_01x01 J105
-U 1 1 5A512B21
-P 10540 2925
-F 0 "J105" H 10540 3025 50  0000 C CNN
-F 1 "Conn_01x01" H 10540 2825 50  0000 C CNN
-F 2 "Connectors:1pin" H 10540 2925 50  0001 C CNN
-F 3 "" H 10540 2925 50  0001 C CNN
-	1    10540 2925
-	1    0    0    -1
-$EndComp
-Wire Wire Line
-	10340 2925 10210 2925
-$Comp
 L Conn_Coaxial J109
 U 1 1 5A5A7286
-P 1620 2755
-F 0 "J109" H 1630 2875 50  0000 C CNN
-F 1 "Conn_Coaxial" V 1735 2755 50  0000 C CNN
-F 2 "rajsradar:132322" H 1620 2755 50  0001 C CNN
-F 3 "" H 1620 2755 50  0001 C CNN
-	1    1620 2755
+P 2785 2755
+F 0 "J109" H 2795 2875 50  0000 C CNN
+F 1 "Conn_Coaxial" V 2900 2755 50  0000 C CNN
+F 2 "rajsradar:132322" H 2785 2755 50  0001 C CNN
+F 3 "" H 2785 2755 50  0001 C CNN
+	1    2785 2755
 	-1   0    0    -1
 $EndComp
@@
 L GND #PWR025
 U 1 1 5A5A8BA4
-P 1620 3045
-F 0 "#PWR025" H 1620 2795 50  0001 C CNN
-F 1 "GND" H 1620 2895 50  0000 C CNN
-F 2 "" H 1620 3045 50  0001 C CNN
-F 3 "" H 1620 3045 50  0001 C CNN
-	1    1620 3045
-	1    0    0    -1
-$EndComp
-Wire Wire Line
-	1620 2955 1620 3045
+P 2785 3045
+F 0 "#PWR025" H 2785 2795 50  0001 C CNN
+F 1 "GND" H 2785 2895 50  0000 C CNN
+F 2 "" H 2785 3045 50  0001 C CNN
+F 3 "" H 2785 3045 50  0001 C CNN
+	1    2785 3045
+	1    0    0    -1
+$EndComp
+Wire Wire Line
+	2785 2955 2785 3045
 $Comp
 L GND #PWR?
@@
 Wire Wire Line
 	1575 2050 1695 2050
+$Comp
+L Conn_01x02 J?
+U 1 1 5AC395BB
+P 10550 2870
+F 0 "J?" H 10550 2970 50  0000 C CNN
+F 1 "Conn_01x02" H 10550 2670 50  0000 C CNN
+F 2 "" H 10550 2870 50  0001 C CNN
+F 3 "" H 10550 2870 50  0001 C CNN
+	1    10550 2870
+	1    0    0    -1
+$EndComp
+Wire Wire Line
+	10210 2870 10350 2870
+Wire Wire Line
+	10350 2970 10210 2970
+Wire Wire Line
+	5990 3305 7795 3305
 $EndSCHEMATC
