File: rf2baseband.sch (KiCad schematic (older format))
At the start: 23 parts

Commit message: Schematic finished
Parts:
- gave numbers to parts that had none: 20
Connections:
- net +12V: now also U701.11; no longer U701.4
- net +6V: now also U701.1, U701.3 (+); no longer U701.1, U701.2 (-)
- net GND: now also U701.4; no longer U701.11
- net at R708.2, R709.1: now also U701.2 (-); no longer U701.3 (+)
- net at R705.2, R707.1: now also U701.10 (+); no longer U701.5 (+)
- net at R701.1, R702.2: now also U701.9 (-); no longer U701.6 (-)
- net at R701.2, R703.1: now also U701.8; no longer U701.7
- net at C704.1, R704.2: now also U701.5 (+); no longer U701.10 (+)
- net at C701.1, C703.1: now also U701.6 (-), U701.7; no longer U701.8, U701.9 (-)
- net at C703.2, R706.1: now also U701.12 (+); no longer U701.12 (+)
- net at RV701.2: now also U701.13 (-); no longer U701.13 (-)
- net at C702.1, RV701.1: now also U701.14; no longer U701.14
Changed lines of the file:
@@
 LIBS:2450bl15b050
 LIBS:tlv4172
+LIBS:l4940d2t12-tr
+LIBS:tps54308
+LIBS:l78l33abu
+LIBS:adp150aujz-18
 LIBS:radar-cache
+LIBS:hn1c01fu
 EELAYER 25 0
 EELAYER END
 $Descr A4 11693 8268
 encoding utf-8
-Sheet 7 7
+Sheet 7 8
 Title ""
 Date ""
@@
 $EndDescr
 $Comp
-L TLV4172 U?
-U 1 1 59DEF024
+L TLV4172 U701
+U 4 1 59DEF024
+P 7140 2460
+F 0 "U701" H 7140 2460 60  0000 C CNN
+F 1 "TLV4172" H 7340 2310 60  0000 C CNN
+F 2 "" H 7140 2460 60  0001 C CNN
+F 3 "" H 7140 2460 60  0001 C CNN
+	4    7140 2460
+	1    0    0    -1
+$EndComp
+$Comp
+L TLV4172 U701
+U 3 1 59DEF055
+P 3540 2660
+F 0 "U701" H 3540 2660 60  0000 C CNN
+F 1 "TLV4172" H 3740 2510 60  0000 C CNN
+F 2 "" H 3540 2660 60  0001 C CNN
+F 3 "" H 3540 2660 60  0001 C CNN
+	3    3540 2660
+	1    0    0    -1
+$EndComp
+$Comp
+L TLV4172 U701
+U 2 1 59DEF098
+P 5330 2560
+F 0 "U701" H 5330 2560 60  0000 C CNN
+F 1 "TLV4172" H 5530 2410 60  0000 C CNN
+F 2 "" H 5330 2560 60  0001 C CNN
+F 3 "" H 5330 2560 60  0001 C CNN
+	2    5330 2560
+	1    0    0    -1
+$EndComp
+$Comp
+L TLV4172 U701
+U 1 1 59DEF0E7
 P 3870 4410
-F 0 "U?" H 3870 4410 60  0000 C CNN
+F 0 "U701" H 3870 4410 60  0000 C CNN
 F 1 "TLV4172" H 4070 4260 60  0000 C CNN
 F 2 "" H 3870 4410 60  0001 C CNN
 F 3 "" H 3870 4410 60  0001 C CNN
 	1    3870 4410
-	1    0    0    -1
-$EndComp
-$Comp
-L TLV4172 U?
-U 2 1 59DEF055
-P 3540 2660
-F 0 "U?" H 3540 2660 60  0000 C CNN
-F 1 "TLV4172" H 3740 2510 60  0000 C CNN
-F 2 "" H 3540 2660 60  0001 C CNN
-F 3 "" H 3540 2660 60  0001 C CNN
-	2    3540 2660
-	1    0    0    -1
-$EndComp
-$Comp
-L TLV4172 U?
-U 3 1 59DEF098
-P 5330 2560
-F 0 "U?" H 5330 2560 60  0000 C CNN
-F 1 "TLV4172" H 5530 2410 60  0000 C CNN
-F 2 "" H 5330 2560 60  0001 C CNN
-F 3 "" H 5330 2560 60  0001 C CNN
-	3    5330 2560
-	1    0    0    -1
-$EndComp
-$Comp
-L TLV4172 U?
-U 4 1 59DEF0E7
-P 7140 2460
-F 0 "U?" H 7140 2460 60  0000 C CNN
-F 1 "TLV4172" H 7340 2310 60  0000 C CNN
-F 2 "" H 7140 2460 60  0001 C CNN
-F 3 "" H 7140 2460 60  0001 C CNN
-	4    7140 2460
-	1    0    0    -1
-$EndComp
-$Comp
-L +12V #PWR?
+	1    0    0    1
+$EndComp
+$Comp
+L +12V #PWR065
 U 1 1 59E0B7DF
 P 3770 3920
-F 0 "#PWR?" H 3770 3770 50  0001 C CNN
+F 0 "#PWR065" H 3770 3770 50  0001 C CNN
 F 1 "+12V" H 3770 4060 50  0000 C CNN
 F 2 "" H 3770 3920 50  0001 C CNN
@@
 	4220 4410 4530 4410
 $Comp
-L R_Small R?
+L R_Small R708
 U 1 1 59E0B935
 P 3250 4340
-F 0 "R?" H 3280 4360 50  0000 L CNN
+F 0 "R708" H 3280 4360 50  0000 L CNN
 F 1 "100k" H 3280 4300 50  0000 L CNN
 F 2 "" H 3250 4340 50  0001 C CNN
@@
 $EndComp
 $Comp
-L R_Small R?
+L R_Small R709
 U 1 1 59E0B9CB
 P 3250 4680
-F 0 "R?" H 3280 4700 50  0000 L CNN
+F 0 "R709" H 3280 4700 50  0000 L CNN
 F 1 "100k" H 3280 4640 50  0000 L CNN
 F 2 "" H 3250 4680 50  0001 C CNN
@@
 $EndComp
 $Comp
-L +12V #PWR?
+L +12V #PWR066
 U 1 1 59E0BA0D
 P 3250 4150
-F 0 "#PWR?" H 3250 4000 50  0001 C CNN
+F 0 "#PWR066" H 3250 4000 50  0001 C CNN
 F 1 "+12V" H 3250 4290 50  0000 C CNN
 F 2 "" H 3250 4150 50  0001 C CNN
@@
 Connection ~ 3250 4510
 $Comp
-L GND #PWR?
+L GND #PWR067
 U 1 1 59E0BA54
 P 3250 4860
-F 0 "#PWR?" H 3250 4610 50  0001 C CNN
+F 0 "#PWR067" H 3250 4610 50  0001 C CNN
 F 1 "GND" H 3250 4710 50  0000 C CNN
 F 2 "" H 3250 4860 50  0001 C CNN
@@
 $EndComp
 $Comp
-L GND #PWR?
+L GND #PWR068
 U 1 1 59E0BA78
 P 3770 4840
-F 0 "#PWR?" H 3770 4590 50  0001 C CNN
+F 0 "#PWR068" H 3770 4590 50  0001 C CNN
 F 1 "GND" H 3770 4690 50  0000 C CNN
 F 2 "" H 3770 4840 50  0001 C CNN
@@
 	3250 4780 3250 4860
 $Comp
-L +6V #PWR?
+L +6V #PWR069
 U 1 1 59E0BD90
 P 4530 4210
-F 0 "#PWR?" H 4530 4060 50  0001 C CNN
+F 0 "#PWR069" H 4530 4060 50  0001 C CNN
 F 1 "+6V" H 4530 4350 50  0000 C CNN
 F 2 "" H 4530 4210 50  0001 C CNN
@@
 Connection ~ 4340 4410
 $Comp
-L R_Small R?
+L R_Small R702
 U 1 1 59E0C2B4
 P 2800 2560
-F 0 "R?" H 2830 2580 50  0000 L CNN
+F 0 "R702" H 2830 2580 50  0000 L CNN
 F 1 "47k" H 2830 2520 50  0000 L CNN
 F 2 "" H 2800 2560 50  0001 C CNN
@@
 $EndComp
 $Comp
-L R_Small R?
+L R_Small R705
 U 1 1 59E0C3CA
 P 2800 2760
-F 0 "R?" H 2830 2780 50  0000 L CNN
+F 0 "R705" H 2830 2780 50  0000 L CNN
 F 1 "47k" H 2830 2720 50  0000 L CNN
 F 2 "" H 2800 2760 50  0001 C CNN
@@
 	3140 2760 2900 2760
 $Comp
-L R_Small R?
+L R_Small R707
 U 1 1 59E0C432
 P 3010 3010
-F 0 "R?" H 3040 3030 50  0000 L CNN
+F 0 "R707" H 3040 3030 50  0000 L CNN
 F 1 "47k" H 3040 2970 50  0000 L CNN
 F 2 "" H 3010 3010 50  0001 C CNN
@@
 $EndComp
 $Comp
-L R_Small R?
+L R_Small R701
 U 1 1 59E0C4FF
 P 3370 2300
-F 0 "R?" H 3400 2320 50  0000 L CNN
+F 0 "R701" H 3400 2320 50  0000 L CNN
 F 1 "47k" H 3400 2260 50  0000 L CNN
 F 2 "" H 3370 2300 50  0001 C CNN
@@
 	2700 2560 2540 2560
 $Comp
-L +6V #PWR?
+L +6V #PWR070
 U 1 1 59E0C944
 P 2740 3110
-F 0 "#PWR?" H 2740 2960 50  0001 C CNN
+F 0 "#PWR070" H 2740 2960 50  0001 C CNN
 F 1 "+6V" H 2740 3250 50  0000 C CNN
 F 2 "" H 2740 3110 50  0001 C CNN
@@
 	3010 3200 3010 3110
 $Comp
-L C_Small C?
+L C_Small C703
 U 1 1 59E0CB5D
 P 6000 2560
-F 0 "C?" H 6010 2630 50  0000 L CNN
+F 0 "C703" H 6010 2630 50  0000 L CNN
 F 1 "1u" H 6010 2480 50  0000 L CNN
 F 2 "" H 6000 2560 50  0001 C CNN
@@
 Connection ~ 4050 2660
 $Comp
-L R_Small R?
+L R_Small R706
 U 1 1 59E0CF2E
 P 6230 2860
-F 0 "R?" H 6260 2880 50  0000 L CNN
+F 0 "R706" H 6260 2880 50  0000 L CNN
 F 1 "100k" H 6260 2820 50  0000 L CNN
 F 2 "" H 6230 2860 50  0001 C CNN
@@
 $EndComp
 $Comp
-L POT RV?
+L POT RV701
 U 1 1 59E0D031
 P 6480 2360
-F 0 "RV?" V 6305 2360 50  0000 C CNN
+F 0 "RV701" V 6305 2360 50  0000 C CNN
 F 1 "1M" V 6380 2360 50  0000 C CNN
 F 2 "" H 6480 2360 50  0001 C CNN
@@
 Connection ~ 6230 2560
 $Comp
-L +6V #PWR?
+L +6V #PWR071
 U 1 1 59E0D23E
 P 6730 2830
-F 0 "#PWR?" H 6730 2680 50  0001 C CNN
+F 0 "#PWR071" H 6730 2680 50  0001 C CNN
 F 1 "+6V" H 6730 2970 50  0000 C CNN
 F 2 "" H 6730 2830 50  0001 C CNN
@@
 	7490 2460 7720 2460
 $Comp
-L R_Small R?
+L R_Small R703
 U 1 1 59E0E057
 P 4350 2660
-F 0 "R?" H 4380 2680 50  0000 L CNN
+F 0 "R703" H 4380 2680 50  0000 L CNN
 F 1 "68k" H 4380 2620 50  0000 L CNN
 F 2 "" H 4350 2660 50  0001 C CNN
@@
 $EndComp
 $Comp
-L R_Small R?
+L R_Small R704
 U 1 1 59E0E10A
 P 4620 2660
-F 0 "R?" H 4650 2680 50  0000 L CNN
+F 0 "R704" H 4650 2680 50  0000 L CNN
 F 1 "68k" H 4650 2620 50  0000 L CNN
 F 2 "" H 4620 2660 50  0001 C CNN
@@
 $EndComp
 $Comp
-L C_Small C?
+L C_Small C704
 U 1 1 59E0E1D3
 P 4840 2960
-F 0 "C?" H 4850 3030 50  0000 L CNN
+F 0 "C704" H 4850 3030 50  0000 L CNN
 F 1 "22p" H 4850 2880 50  0000 L CNN
 F 2 "" H 4840 2960 50  0001 C CNN
@@
 $EndComp
 $Comp
-L C_Small C?
+L C_Small C701
 U 1 1 59E0E272
 P 5080 2000
-F 0 "C?" H 5090 2070 50  0000 L CNN
+F 0 "C701" H 5090 2070 50  0000 L CNN
 F 1 "22p" H 5090 1920 50  0000 L CNN
 F 2 "" H 5080 2000 50  0001 C CNN
@@
 Connection ~ 5800 2230
 $Comp
-L +6V #PWR?
+L +6V #PWR072
 U 1 1 59E0E4F0
 P 5280 3020
-F 0 "#PWR?" H 5280 2870 50  0001 C CNN
+F 0 "#PWR072" H 5280 2870 50  0001 C CNN
 F 1 "+6V" H 5280 3160 50  0000 C CNN
 F 2 "" H 5280 3020 50  0001 C CNN
@@
 	4840 3200 4840 3060
 $Comp
-L C_Small C?
+L C_Small C702
 U 1 1 59E0E7CF
 P 7820 2460
-F 0 "C?" H 7830 2530 50  0000 L CNN
+F 0 "C702" H 7830 2530 50  0000 L CNN
 F 1 "1u" H 7830 2380 50  0000 L CNN
 F 2 "" H 7820 2460 50  0001 C CNN
@@
 100kHz LPF
 $Comp
-L +12V #PWR?
+L +12V #PWR073
 U 1 1 59E1133D
 P 6880 4110
-F 0 "#PWR?" H 6880 3960 50  0001 C CNN
+F 0 "#PWR073" H 6880 3960 50  0001 C CNN
 F 1 "+12V" H 6880 4250 50  0000 C CNN
 F 2 "" H 6880 4110 50  0001 C CNN
@@
 $EndComp
 $Comp
-L C_Small C?
+L C_Small C706
 U 1 1 59E11387
 P 6460 4310
-F 0 "C?" H 6470 4380 50  0000 L CNN
+F 0 "C706" H 6470 4380 50  0000 L CNN
 F 1 "10u" H 6470 4230 50  0000 L CNN
 F 2 "" H 6460 4310 50  0001 C CNN
@@
 $EndComp
 $Comp
-L C_Small C?
+L C_Small C705
 U 1 1 59E1149D
 P 6250 4310
-F 0 "C?" H 6260 4380 50  0000 L CNN
+F 0 "C705" H 6260 4380 50  0000 L CNN
 F 1 "22u" H 6260 4230 50  0000 L CNN
 F 2 "" H 6250 4310 50  0001 C CNN
@@
 $EndComp
 $Comp
-L C_Small C?
+L C_Small C707
 U 1 1 59E11519
 P 6680 4310
-F 0 "C?" H 6690 4380 50  0000 L CNN
+F 0 "C707" H 6690 4380 50  0000 L CNN
 F 1 "1u" H 6690 4230 50  0000 L CNN
 F 2 "" H 6680 4310 50  0001 C CNN
@@
 $EndComp
 $Comp
-L C_Small C?
+L C_Small C708
 U 1 1 59E1158A
 P 6880 4310
-F 0 "C?" H 6890 4380 50  0000 L CNN
+F 0 "C708" H 6890 4380 50  0000 L CNN
 F 1 "100n" H 6890 4230 50  0000 L CNN
 F 2 "" H 6880 4310 50  0001 C CNN
@@
 $EndComp
 $Comp
-L +12VA #PWR?
+L +12VA #PWR074
 U 1 1 59E119E6
 P 6250 3810
-F 0 "#PWR?" H 6250 3660 50  0001 C CNN
+F 0 "#PWR074" H 6250 3660 50  0001 C CNN
 F 1 "+12VA" H 6250 3950 50  0000 C CNN
 F 2 "" H 6250 3810 50  0001 C CNN
@@
 Connection ~ 6680 4160
 $Comp
-L GND #PWR?
+L GND #PWR075
 U 1 1 59E1200C
 P 6250 4470
-F 0 "#PWR?" H 6250 4220 50  0001 C CNN
+F 0 "#PWR075" H 6250 4220 50  0001 C CNN
 F 1 "GND" H 6250 4320 50  0000 C CNN
 F 2 "" H 6250 4470 50  0001 C CNN
@@
 $EndComp
 $Comp
-L GND #PWR?
+L GND #PWR076
 U 1 1 59E12063
 P 6460 4470
-F 0 "#PWR?" H 6460 4220 50  0001 C CNN
+F 0 "#PWR076" H 6460 4220 50  0001 C CNN
 F 1 "GND" H 6460 4320 50  0000 C CNN
 F 2 "" H 6460 4470 50  0001 C CNN
@@
 $EndComp
 $Comp
-L GND #PWR?
+L GND #PWR077
 U 1 1 59E120B3
 P 6680 4470
-F 0 "#PWR?" H 6680 4220 50  0001 C CNN
+F 0 "#PWR077" H 6680 4220 50  0001 C CNN
 F 1 "GND" H 6680 4320 50  0000 C CNN
 F 2 "" H 6680 4470 50  0001 C CNN
@@
 $EndComp
 $Comp
-L GND #PWR?
+L GND #PWR078
 U 1 1 59E12103
 P 6880 4470
-F 0 "#PWR?" H 6880 4220 50  0001 C CNN
+F 0 "#PWR078" H 6880 4220 50  0001 C CNN
 F 1 "GND" H 6880 4320 50  0000 C CNN
 F 2 "" H 6880 4470 50  0001 C CNN
@@
 	6880 4410 6880 4470
 $Comp
-L L_Core_Ferrite_Small L?
+L L_Core_Ferrite_Small L701
 U 1 1 59E16A96
 P 6250 4000
-F 0 "L?" H 6300 4040 50  0000 L CNN
+F 0 "L701" H 6300 4040 50  0000 L CNN
 F 1 "L_Core_Ferrite_Small" H 6300 3950 50  0000 L CNN
 F 2 "" H 6250 4000 50  0001 C CNN

Commit message: Assign a lot of footprints, fix l78l33abu part (input and output were reversed)
Parts:
- C701, C702, C703, C704, C707, C708: footprint (none) -> Capacitors_SMD:C_0603_HandSoldering
- C705: footprint (none) -> Capacitors_SMD:C_1210_HandSoldering
- C706: footprint (none) -> Capacitors_SMD:C_0805_HandSoldering
- R701, R702, R705, R707: footprint (none) -> Resistors_SMD:R_0603_HandSoldering
- R703, R704: footprint (none) -> Resistors_SMD:R_1206_HandSoldering
- R706, R708, R709: footprint (none) -> Resistors_SMD:R_0402
- U701: footprint (none) -> Housings_SSOP:TSSOP-14_4.4x5mm_Pitch0.65mm
Changed lines of the file:
@@
 F 0 "U701" H 7140 2460 60  0000 C CNN
 F 1 "TLV4172" H 7340 2310 60  0000 C CNN
-F 2 "" H 7140 2460 60  0001 C CNN
+F 2 "Housings_SSOP:TSSOP-14_4.4x5mm_Pitch0.65mm" H 7140 2460 60  0001 C CNN
 F 3 "" H 7140 2460 60  0001 C CNN
 	4    7140 2460
@@
 F 0 "U701" H 3540 2660 60  0000 C CNN
 F 1 "TLV4172" H 3740 2510 60  0000 C CNN
-F 2 "" H 3540 2660 60  0001 C CNN
+F 2 "Housings_SSOP:TSSOP-14_4.4x5mm_Pitch0.65mm" H 3540 2660 60  0001 C CNN
 F 3 "" H 3540 2660 60  0001 C CNN
 	3    3540 2660
@@
 F 0 "U701" H 5330 2560 60  0000 C CNN
 F 1 "TLV4172" H 5530 2410 60  0000 C CNN
-F 2 "" H 5330 2560 60  0001 C CNN
+F 2 "Housings_SSOP:TSSOP-14_4.4x5mm_Pitch0.65mm" H 5330 2560 60  0001 C CNN
 F 3 "" H 5330 2560 60  0001 C CNN
 	2    5330 2560
@@
 F 0 "U701" H 3870 4410 60  0000 C CNN
 F 1 "TLV4172" H 4070 4260 60  0000 C CNN
-F 2 "" H 3870 4410 60  0001 C CNN
+F 2 "Housings_SSOP:TSSOP-14_4.4x5mm_Pitch0.65mm" H 3870 4410 60  0001 C CNN
 F 3 "" H 3870 4410 60  0001 C CNN
 	1    3870 4410
@@
 $EndComp
 $Comp
-L +12V #PWR065
+L +12V #PWR066
 U 1 1 59E0B7DF
 P 3770 3920
-F 0 "#PWR065" H 3770 3770 50  0001 C CNN
+F 0 "#PWR066" H 3770 3770 50  0001 C CNN
 F 1 "+12V" H 3770 4060 50  0000 C CNN
 F 2 "" H 3770 3920 50  0001 C CNN
@@
 F 0 "R708" H 3280 4360 50  0000 L CNN
 F 1 "100k" H 3280 4300 50  0000 L CNN
-F 2 "" H 3250 4340 50  0001 C CNN
+F 2 "Resistors_SMD:R_0402" H 3250 4340 50  0001 C CNN
 F 3 "" H 3250 4340 50  0001 C CNN
 	1    3250 4340
@@
 F 0 "R709" H 3280 4700 50  0000 L CNN
 F 1 "100k" H 3280 4640 50  0000 L CNN
-F 2 "" H 3250 4680 50  0001 C CNN
+F 2 "Resistors_SMD:R_0402" H 3250 4680 50  0001 C CNN
 F 3 "" H 3250 4680 50  0001 C CNN
 	1    3250 4680
@@
 $EndComp
 $Comp
-L +12V #PWR066
+L +12V #PWR067
 U 1 1 59E0BA0D
 P 3250 4150
-F 0 "#PWR066" H 3250 4000 50  0001 C CNN
+F 0 "#PWR067" H 3250 4000 50  0001 C CNN
 F 1 "+12V" H 3250 4290 50  0000 C CNN
 F 2 "" H 3250 4150 50  0001 C CNN
@@
 Connection ~ 3250 4510
 $Comp
-L GND #PWR067
+L GND #PWR068
 U 1 1 59E0BA54
 P 3250 4860
-F 0 "#PWR067" H 3250 4610 50  0001 C CNN
+F 0 "#PWR068" H 3250 4610 50  0001 C CNN
 F 1 "GND" H 3250 4710 50  0000 C CNN
 F 2 "" H 3250 4860 50  0001 C CNN
@@
 $EndComp
 $Comp
-L GND #PWR068
+L GND #PWR069
 U 1 1 59E0BA78
 P 3770 4840
-F 0 "#PWR068" H 3770 4590 50  0001 C CNN
+F 0 "#PWR069" H 3770 4590 50  0001 C CNN
 F 1 "GND" H 3770 4690 50  0000 C CNN
 F 2 "" H 3770 4840 50  0001 C CNN
@@
 	3250 4780 3250 4860
 $Comp
-L +6V #PWR069
+L +6V #PWR070
 U 1 1 59E0BD90
 P 4530 4210
-F 0 "#PWR069" H 4530 4060 50  0001 C CNN
+F 0 "#PWR070" H 4530 4060 50  0001 C CNN
 F 1 "+6V" H 4530 4350 50  0000 C CNN
 F 2 "" H 4530 4210 50  0001 C CNN
@@
 F 0 "R702" H 2830 2580 50  0000 L CNN
 F 1 "47k" H 2830 2520 50  0000 L CNN
-F 2 "" H 2800 2560 50  0001 C CNN
+F 2 "Resistors_SMD:R_0603_HandSoldering" H 2800 2560 50  0001 C CNN
 F 3 "" H 2800 2560 50  0001 C CNN
 	1    2800 2560
@@
 F 0 "R705" H 2830 2780 50  0000 L CNN
 F 1 "47k" H 2830 2720 50  0000 L CNN
-F 2 "" H 2800 2760 50  0001 C CNN
+F 2 "Resistors_SMD:R_0603_HandSoldering" H 2800 2760 50  0001 C CNN
 F 3 "" H 2800 2760 50  0001 C CNN
 	1    2800 2760
@@
 F 0 "R707" H 3040 3030 50  0000 L CNN
 F 1 "47k" H 3040 2970 50  0000 L CNN
-F 2 "" H 3010 3010 50  0001 C CNN
+F 2 "Resistors_SMD:R_0603_HandSoldering" H 3010 3010 50  0001 C CNN
 F 3 "" H 3010 3010 50  0001 C CNN
 	1    3010 3010
@@
 F 0 "R701" H 3400 2320 50  0000 L CNN
 F 1 "47k" H 3400 2260 50  0000 L CNN
-F 2 "" H 3370 2300 50  0001 C CNN
+F 2 "Resistors_SMD:R_0603_HandSoldering" H 3370 2300 50  0001 C CNN
 F 3 "" H 3370 2300 50  0001 C CNN
 	1    3370 2300
@@
 	2700 2560 2540 2560
 $Comp
-L +6V #PWR070
+L +6V #PWR071
 U 1 1 59E0C944
 P 2740 3110
-F 0 "#PWR070" H 2740 2960 50  0001 C CNN
+F 0 "#PWR071" H 2740 2960 50  0001 C CNN
 F 1 "+6V" H 2740 3250 50  0000 C CNN
 F 2 "" H 2740 3110 50  0001 C CNN
@@
 F 0 "C703" H 6010 2630 50  0000 L CNN
 F 1 "1u" H 6010 2480 50  0000 L CNN
-F 2 "" H 6000 2560 50  0001 C CNN
+F 2 "Capacitors_SMD:C_0603_HandSoldering" H 6000 2560 50  0001 C CNN
 F 3 "" H 6000 2560 50  0001 C CNN
 	1    6000 2560
@@
 F 0 "R706" H 6260 2880 50  0000 L CNN
 F 1 "100k" H 6260 2820 50  0000 L CNN
-F 2 "" H 6230 2860 50  0001 C CNN
+F 2 "Resistors_SMD:R_0402" H 6230 2860 50  0001 C CNN
 F 3 "" H 6230 2860 50  0001 C CNN
 	1    6230 2860
@@
 Connection ~ 6230 2560
 $Comp
-L +6V #PWR071
+L +6V #PWR072
 U 1 1 59E0D23E
 P 6730 2830
-F 0 "#PWR071" H 6730 2680 50  0001 C CNN
+F 0 "#PWR072" H 6730 2680 50  0001 C CNN
 F 1 "+6V" H 6730 2970 50  0000 C CNN
 F 2 "" H 6730 2830 50  0001 C CNN
@@
 F 0 "R703" H 4380 2680 50  0000 L CNN
 F 1 "68k" H 4380 2620 50  0000 L CNN
-F 2 "" H 4350 2660 50  0001 C CNN
+F 2 "Resistors_SMD:R_1206_HandSoldering" H 4350 2660 50  0001 C CNN
 F 3 "" H 4350 2660 50  0001 C CNN
 	1    4350 2660
@@
 F 0 "R704" H 4650 2680 50  0000 L CNN
 F 1 "68k" H 4650 2620 50  0000 L CNN
-F 2 "" H 4620 2660 50  0001 C CNN
+F 2 "Resistors_SMD:R_1206_HandSoldering" H 4620 2660 50  0001 C CNN
 F 3 "" H 4620 2660 50  0001 C CNN
 	1    4620 2660
@@
 F 0 "C704" H 4850 3030 50  0000 L CNN
 F 1 "22p" H 4850 2880 50  0000 L CNN
-F 2 "" H 4840 2960 50  0001 C CNN
+F 2 "Capacitors_SMD:C_0603_HandSoldering" H 4840 2960 50  0001 C CNN
 F 3 "" H 4840 2960 50  0001 C CNN
 	1    4840 2960
@@
 F 0 "C701" H 5090 2070 50  0000 L CNN
 F 1 "22p" H 5090 1920 50  0000 L CNN
-F 2 "" H 5080 2000 50  0001 C CNN
+F 2 "Capacitors_SMD:C_0603_HandSoldering" H 5080 2000 50  0001 C CNN
 F 3 "" H 5080 2000 50  0001 C CNN
 	1    5080 2000
@@
 Connection ~ 5800 2230
 $Comp
-L +6V #PWR072
+L +6V #PWR073
 U 1 1 59E0E4F0
 P 5280 3020
-F 0 "#PWR072" H 5280 2870 50  0001 C CNN
+F 0 "#PWR073" H 5280 2870 50  0001 C CNN
 F 1 "+6V" H 5280 3160 50  0000 C CNN
 F 2 "" H 5280 3020 50  0001 C CNN
@@
 F 0 "C702" H 7830 2530 50  0000 L CNN
 F 1 "1u" H 7830 2380 50  0000 L CNN
-F 2 "" H 7820 2460 50  0001 C CNN
+F 2 "Capacitors_SMD:C_0603_HandSoldering" H 7820 2460 50  0001 C CNN
 F 3 "" H 7820 2460 50  0001 C CNN
 	1    7820 2460
@@
 100kHz LPF
 $Comp
-L +12V #PWR073
+L +12V #PWR074
 U 1 1 59E1133D
 P 6880 4110
-F 0 "#PWR073" H 6880 3960 50  0001 C CNN
+F 0 "#PWR074" H 6880 3960 50  0001 C CNN
 F 1 "+12V" H 6880 4250 50  0000 C CNN
 F 2 "" H 6880 4110 50  0001 C CNN
@@
 F 0 "C706" H 6470 4380 50  0000 L CNN
 F 1 "10u" H 6470 4230 50  0000 L CNN
-F 2 "" H 6460 4310 50  0001 C CNN
+F 2 "Capacitors_SMD:C_0805_HandSoldering" H 6460 4310 50  0001 C CNN
 F 3 "" H 6460 4310 50  0001 C CNN
 	1    6460 4310
@@
 F 0 "C705" H 6260 4380 50  0000 L CNN
 F 1 "22u" H 6260 4230 50  0000 L CNN
-F 2 "" H 6250 4310 50  0001 C CNN
+F 2 "Capacitors_SMD:C_1210_HandSoldering" H 6250 4310 50  0001 C CNN
 F 3 "" H 6250 4310 50  0001 C CNN
 	1    6250 4310
@@
 F 0 "C707" H 6690 4380 50  0000 L CNN
 F 1 "1u" H 6690 4230 50  0000 L CNN
-F 2 "" H 6680 4310 50  0001 C CNN
+F 2 "Capacitors_SMD:C_0603_HandSoldering" H 6680 4310 50  0001 C CNN
 F 3 "" H 6680 4310 50  0001 C CNN
 	1    6680 4310
@@
 F 0 "C708" H 6890 4380 50  0000 L CNN
 F 1 "100n" H 6890 4230 50  0000 L CNN
-F 2 "" H 6880 4310 50  0001 C CNN
+F 2 "Capacitors_SMD:C_0603_HandSoldering" H 6880 4310 50  0001 C CNN
 F 3 "" H 6880 4310 50  0001 C CNN
 	1    6880 4310
@@
 $EndComp
 $Comp
-L +12VA #PWR074
+L +12VA #PWR075
 U 1 1 59E119E6
 P 6250 3810
-F 0 "#PWR074" H 6250 3660 50  0001 C CNN
+F 0 "#PWR075" H 6250 3660 50  0001 C CNN
 F 1 "+12VA" H 6250 3950 50  0000 C CNN
 F 2 "" H 6250 3810 50  0001 C CNN
@@
 Connection ~ 6680 4160
 $Comp
-L GND #PWR075
+L GND #PWR076
 U 1 1 59E1200C
 P 6250 4470
-F 0 "#PWR075" H 6250 4220 50  0001 C CNN
+F 0 "#PWR076" H 6250 4220 50  0001 C CNN
 F 1 "GND" H 6250 4320 50  0000 C CNN
 F 2 "" H 6250 4470 50  0001 C CNN
@@
 $EndComp
 $Comp
-L GND #PWR076
+L GND #PWR077
 U 1 1 59E12063
 P 6460 4470
-F 0 "#PWR076" H 6460 4220 50  0001 C CNN
+F 0 "#PWR077" H 6460 4220 50  0001 C CNN
 F 1 "GND" H 6460 4320 50  0000 C CNN
 F 2 "" H 6460 4470 50  0001 C CNN
@@
 $EndComp
 $Comp
-L GND #PWR077
+L GND #PWR078
 U 1 1 59E120B3
 P 6680 4470
-F 0 "#PWR077" H 6680 4220 50  0001 C CNN
+F 0 "#PWR078" H 6680 4220 50  0001 C CNN
 F 1 "GND" H 6680 4320 50  0000 C CNN
 F 2 "" H 6680 4470 50  0001 C CNN
@@
 $EndComp
 $Comp
-L GND #PWR078
+L GND #PWR079
 U 1 1 59E12103
 P 6880 4470
-F 0 "#PWR078" H 6880 4220 50  0001 C CNN
+F 0 "#PWR079" H 6880 4220 50  0001 C CNN
 F 1 "GND" H 6880 4320 50  0000 C CNN
 F 2 "" H 6880 4470 50  0001 C CNN
