File: rf/levelshifter.sch (KiCad schematic (older format))
At the start: 2 parts, among them U801 SN74LV1T34, U802 SN74LV1T34

Commit message: Finish first revision layout
Parts:
- renumbered U801 to U701, U802 to U702
Changed lines of the file:
@@
 LIBS:mc2016k30
 LIBS:cp0402q5425entr
+LIBS:lm340-5
 EELAYER 25 0
 EELAYER END
@@
 	7390 3615 7190 3615
 $Comp
-L SN74LV1T34 U801
+L SN74LV1T34 U701
 U 1 1 5A7E7EF8
 P 4790 3715
-F 0 "U801" H 4790 3715 60  0000 C CNN
+F 0 "U701" H 4790 3715 60  0000 C CNN
 F 1 "SN74LV1T34" H 4790 3965 60  0000 C CNN
 F 2 "TO_SOT_Packages_SMD:SOT-23-5_HandSoldering" H 4790 3715 60  0001 C CNN
@@
 $EndComp
 $Comp
-L SN74LV1T34 U802
+L SN74LV1T34 U702
 U 1 1 5A7E7FA3
 P 6890 3715
-F 0 "U802" H 6890 3715 60  0000 C CNN
+F 0 "U702" H 6890 3715 60  0000 C CNN
 F 1 "SN74LV1T34" H 6890 3965 60  0000 C CNN
 F 2 "TO_SOT_Packages_SMD:SOT-23-5_HandSoldering" H 6890 3715 60  0001 C CNN
