File: rf/mixer.sch (KiCad schematic (older format))
At the start: 25 parts, among them T502 2450BL15B100, T504 2450BL15B050, U501 AD8343

Commit message: Finish assigning component footprints
Parts:
- C506, C508: value 1p35 -> 1p3
- C509, C510: value 10n -> 75p
- L501: value 2.5n -> 2.6nH
Changed lines of the file:
@@
 $EndComp
 $Comp
-L GND #PWR043
+L GND #PWR407
 U 1 1 59D5980B
 P 3670 3140
-F 0 "#PWR043" H 3670 2890 50  0001 C CNN
+F 0 "#PWR407" H 3670 2890 50  0001 C CNN
 F 1 "GND" H 3670 2990 50  0000 C CNN
 F 2 "" H 3670 3140 50  0001 C CNN
@@
 $EndComp
 $Comp
-L GND #PWR044
+L GND #PWR408
 U 1 1 59D5982F
 P 3390 3770
-F 0 "#PWR044" H 3390 3520 50  0001 C CNN
+F 0 "#PWR408" H 3390 3520 50  0001 C CNN
 F 1 "GND" H 3390 3620 50  0000 C CNN
 F 2 "" H 3390 3770 50  0001 C CNN
@@
 P 3720 3540
 F 0 "L501" H 3750 3580 50  0000 L CNN
-F 1 "2.5n" H 3750 3500 50  0000 L CNN
+F 1 "2.6nH" H 3750 3500 50  0000 L CNN
 F 2 "Capacitors_SMD:C_0201" H 3720 3540 50  0001 C CNN
 F 3 "" H 3720 3540 50  0001 C CNN
@@
 P 3920 3400
 F 0 "C506" H 3930 3470 50  0000 L CNN
-F 1 "1p35" H 3930 3320 50  0000 L CNN
+F 1 "1p3" H 3930 3320 50  0000 L CNN
 F 2 "Capacitors_SMD:C_0201" H 3920 3400 50  0001 C CNN
 F 3 "" H 3920 3400 50  0001 C CNN
@@
 P 3910 3680
 F 0 "C508" H 3920 3750 50  0000 L CNN
-F 1 "1p35" H 3920 3600 50  0000 L CNN
+F 1 "1p3" H 3920 3600 50  0000 L CNN
 F 2 "Capacitors_SMD:C_0201" H 3910 3680 50  0001 C CNN
 F 3 "" H 3910 3680 50  0001 C CNN
@@
 $EndComp
 $Comp
-L GND #PWR045
+L GND #PWR414
 U 1 1 59D59D07
 P 6040 4480
-F 0 "#PWR045" H 6040 4230 50  0001 C CNN
+F 0 "#PWR414" H 6040 4230 50  0001 C CNN
 F 1 "GND" H 6040 4330 50  0000 C CNN
 F 2 "" H 6040 4480 50  0001 C CNN
@@
 $EndComp
 $Comp
-L GND #PWR046
+L GND #PWR412
 U 1 1 59D5A4DD
 P 4240 4360
-F 0 "#PWR046" H 4240 4110 50  0001 C CNN
+F 0 "#PWR412" H 4240 4110 50  0001 C CNN
 F 1 "GND" H 4240 4210 50  0000 C CNN
 F 2 "" H 4240 4360 50  0001 C CNN
@@
 $EndComp
 $Comp
-L GND #PWR047
+L GND #PWR413
 U 1 1 59D5A52E
 P 4390 4360
-F 0 "#PWR047" H 4390 4110 50  0001 C CNN
+F 0 "#PWR413" H 4390 4110 50  0001 C CNN
 F 1 "GND" H 4390 4210 50  0000 C CNN
 F 2 "" H 4390 4360 50  0001 C CNN
@@
 $EndComp
 $Comp
-L GND #PWR048
+L GND #PWR410
 U 1 1 59D5CBC6
 P 5250 4310
-F 0 "#PWR048" H 5250 4060 50  0001 C CNN
+F 0 "#PWR410" H 5250 4060 50  0001 C CNN
 F 1 "GND" H 5250 4160 50  0000 C CNN
 F 2 "" H 5250 4310 50  0001 C CNN
@@
 $EndComp
 $Comp
-L GND #PWR049
+L GND #PWR411
 U 1 1 59D5CBFC
 P 4860 4320
-F 0 "#PWR049" H 4860 4070 50  0001 C CNN
+F 0 "#PWR411" H 4860 4070 50  0001 C CNN
 F 1 "GND" H 4860 4170 50  0000 C CNN
 F 2 "" H 4860 4320 50  0001 C CNN
@@
 $EndComp
 $Comp
-L +5V #PWR050
+L +5V #PWR404
 U 1 1 59D5CE3D
 P 4600 2580
-F 0 "#PWR050" H 4600 2430 50  0001 C CNN
+F 0 "#PWR404" H 4600 2430 50  0001 C CNN
 F 1 "+5V" H 4600 2720 50  0000 C CNN
 F 2 "" H 4600 2580 50  0001 C CNN
@@
 $EndComp
 $Comp
-L GND #PWR051
+L GND #PWR409
 U 1 1 59D5ED7D
 P 8230 3970
-F 0 "#PWR051" H 8230 3720 50  0001 C CNN
+F 0 "#PWR409" H 8230 3720 50  0001 C CNN
 F 1 "GND" H 8230 3820 50  0000 C CNN
 F 2 "" H 8230 3970 50  0001 C CNN
@@
 P 7040 3800
 F 0 "C510" H 7050 3870 50  0000 L CNN
-F 1 "10n" H 7050 3720 50  0000 L CNN
+F 1 "75p" H 7050 3720 50  0000 L CNN
 F 2 "Capacitors_SMD:C_0402" H 7040 3800 50  0001 C CNN
 F 3 "" H 7040 3800 50  0001 C CNN
@@
 P 7140 3700
 F 0 "C509" H 7150 3770 50  0000 L CNN
-F 1 "10n" H 7150 3620 50  0000 L CNN
+F 1 "75p" H 7150 3620 50  0000 L CNN
 F 2 "Capacitors_SMD:C_0402" H 7140 3700 50  0001 C CNN
 F 3 "" H 7140 3700 50  0001 C CNN
@@
 $EndComp
 $Comp
-L GND #PWR052
+L GND #PWR405
 U 1 1 59D60664
 P 4600 3090
-F 0 "#PWR052" H 4600 2840 50  0001 C CNN
+F 0 "#PWR405" H 4600 2840 50  0001 C CNN
 F 1 "GND" H 4600 2940 50  0000 C CNN
 F 2 "" H 4600 3090 50  0001 C CNN
@@
 $EndComp
 $Comp
-L GND #PWR053
+L GND #PWR406
 U 1 1 59D606AF
 P 4950 3090
-F 0 "#PWR053" H 4950 2840 50  0001 C CNN
+F 0 "#PWR406" H 4950 2840 50  0001 C CNN
 F 1 "GND" H 4950 2940 50  0000 C CNN
 F 2 "" H 4950 3090 50  0001 C CNN
@@
 	5110 3300 5390 3300
 $Comp
-L +5V #PWR054
+L +5V #PWR401
 U 1 1 59D61273
 P 6220 2040
-F 0 "#PWR054" H 6220 1890 50  0001 C CNN
+F 0 "#PWR401" H 6220 1890 50  0001 C CNN
 F 1 "+5V" H 6220 2180 50  0000 C CNN
 F 2 "" H 6220 2040 50  0001 C CNN
@@
 $EndComp
 $Comp
-L GND #PWR055
+L GND #PWR402
 U 1 1 59D6128B
 P 6220 2550
-F 0 "#PWR055" H 6220 2300 50  0001 C CNN
+F 0 "#PWR402" H 6220 2300 50  0001 C CNN
 F 1 "GND" H 6220 2400 50  0000 C CNN
 F 2 "" H 6220 2550 50  0001 C CNN
@@
 $EndComp
 $Comp
-L GND #PWR056
+L GND #PWR403
 U 1 1 59D61291
 P 6570 2550
-F 0 "#PWR056" H 6570 2300 50  0001 C CNN
+F 0 "#PWR403" H 6570 2300 50  0001 C CNN
 F 1 "GND" H 6570 2400 50  0000 C CNN
 F 2 "" H 6570 2550 50  0001 C CNN

Commit message: Finish first revision layout
Parts:
- renumbered C501 to C401, C502 to C402, C503 to C403, C504 to C404, C505 to C405, C506 to C406, C507 to C407, C508 to C408, C509 to C409, C510 to C410, C511 to C411, L501 to L401, L502 to L402, L503 to L403, R501 to R401, R502 to R402, R503 to R403, R504 to R404, R505 to R405, R506 to R406, R507 to R407, R508 to R408, T502 to T401, T504 to T402, U501 to U401
Connections:
- net at T402.3: now also C409.1; no longer C410.1
- net at T402.4: now also C410.1; no longer C409.1
