File: rf/pa.sch (KiCad schematic (older format))
At the start: 8 parts, among them U401 QPA5219

Commit message: Finish first revision layout
Parts:
- renumbered C401 to C301, C402 to C302, C403 to C303, C404 to C304, C405 to C305, R401 to R301, R402 to R302, U401 to U301
Changed lines of the file:
@@
 LIBS:mc2016k30
 LIBS:cp0402q5425entr
+LIBS:lm340-5
 EELAYER 25 0
 EELAYER END
@@
 $EndDescr
 $Comp
-L QPA5219 U401
+L QPA5219 U301
 U 1 1 59D558DD
 P 5460 3360
-F 0 "U401" H 5960 2810 60  0000 C CNN
+F 0 "U301" H 5960 2810 60  0000 C CNN
 F 1 "QPA5219" H 5860 3860 60  0000 C CNN
 F 2 "rajsradar:QPA5219" H 5410 3360 60  0001 C CNN
@@
 $EndComp
 $Comp
-L C_Small C404
+L C_Small C304
 U 1 1 59D55C69
 P 6410 2470
-F 0 "C404" H 6420 2540 50  0000 L CNN
+F 0 "C304" H 6420 2540 50  0000 L CNN
 F 1 "0u1" H 6420 2390 50  0000 L CNN
 F 2 "Capacitors_SMD:C_0603_HandSoldering" H 6410 2470 50  0001 C CNN
@@
 $EndComp
 $Comp
-L C_Small C405
+L C_Small C305
 U 1 1 59D55E73
 P 4810 2640
-F 0 "C405" H 4820 2710 50  0000 L CNN
+F 0 "C305" H 4820 2710 50  0000 L CNN
 F 1 "2u2" H 4820 2560 50  0000 L CNN
 F 2 "Capacitors_SMD:C_0805_HandSoldering" H 4810 2640 50  0001 C CNN
@@
 $EndComp
 $Comp
-L C_Small C401
+L C_Small C301
 U 1 1 59D56103
 P 6410 1790
-F 0 "C401" H 6420 1860 50  0000 L CNN
+F 0 "C301" H 6420 1860 50  0000 L CNN
 F 1 "0u1" H 6420 1710 50  0000 L CNN
 F 2 "Capacitors_SMD:C_0603_HandSoldering" H 6410 1790 50  0001 C CNN
@@
 $EndComp
 $Comp
-L C_Small C402
+L C_Small C302
 U 1 1 59D562A6
 P 6160 1800
-F 0 "C402" H 6170 1870 50  0000 L CNN
+F 0 "C302" H 6170 1870 50  0000 L CNN
 F 1 "2u2" H 6170 1720 50  0000 L CNN
 F 2 "Capacitors_SMD:C_0805_HandSoldering" H 6160 1800 50  0001 C CNN
@@
 $EndComp
 $Comp
-L C_Small C403
+L C_Small C303
 U 1 1 59D5637B
 P 6150 2470
-F 0 "C403" H 6160 2540 50  0000 L CNN
+F 0 "C303" H 6160 2540 50  0000 L CNN
 F 1 "2u2" H 6160 2390 50  0000 L CNN
 F 2 "Capacitors_SMD:C_0805_HandSoldering" H 6150 2470 50  0001 C CNN
@@
 EN
 $Comp
-L R_Small R401
+L R_Small R301
 U 1 1 59D56957
 P 4630 3090
-F 0 "R401" H 4660 3110 50  0000 L CNN
+F 0 "R301" H 4660 3110 50  0000 L CNN
 F 1 "10k" H 4660 3050 50  0000 L CNN
 F 2 "Resistors_SMD:R_0603_HandSoldering" H 4630 3090 50  0001 C CNN
@@
 Connection ~ 4810 2420
 $Comp
-L R_Small R402
+L R_Small R302
 U 1 1 59D57058
 P 6520 3810
-F 0 "R402" H 6550 3830 50  0000 L CNN
+F 0 "R302" H 6550 3830 50  0000 L CNN
 F 1 "27k" H 6550 3770 50  0000 L CNN
 F 2 "Resistors_SMD:R_0603_HandSoldering" H 6520 3810 50  0001 C CNN
