File: rf/vco.sch (KiCad schematic (older format))
At the start: 24 parts, among them U201 MAX2750

Commit message: Finish assigning component footprints
Parts:
- C201, C204, C206, C208, C210: renamed from C?; footprint (none) -> Capacitors_SMD:C_0603_HandSoldering
- C205, C207, C211: renamed from C?; footprint (none) -> Capacitors_SMD:C_0805_HandSoldering
- C209: renamed from C?; footprint (none) -> Capacitors_SMD:C_0402
- C212, C213: renamed from C?; value 100p -> 75p; footprint (none) -> Capacitors_SMD:C_0402
- R202: renamed from R?; footprint (none) -> Resistors_SMD:R_0603_HandSoldering
- R203, R204, R207: renamed from R?; footprint (none) -> Resistors_SMD:R_0402
- R205: renamed from R?; value 137.6 -> 133; footprint (none) -> Resistors_SMD:R_0805_HandSoldering
- R206: renamed from R?; footprint (none) -> Capacitors_SMD:C_0402
- R208: renamed from R?; value 4k7 -> 10k; footprint (none) -> Resistors_SMD:R_0603_HandSoldering
- U202: renamed from U?; footprint (none) -> rajsradar:MC2016K30.0000C16ESH
- U203: renamed from U?; footprint (none) -> rajsradar:TSSOP-16

Commit message: Finish first revision layout
Parts:
- renumbered C202 to C201, C203 to C202, C201 to C203
Connections:
- net GND: now also C201.2, C202.2, C208.2, C210.2, C211.2
Changed lines of the file:
@@
 LIBS:mc2016k30
 LIBS:cp0402q5425entr
+LIBS:lm340-5
 EELAYER 25 0
 EELAYER END
@@
 $EndComp
 $Comp
-L C_Small C203
+L C_Small C202
 U 1 1 59D54372
 P 7630 2615
-F 0 "C203" H 7640 2685 50  0000 L CNN
+F 0 "C202" H 7640 2685 50  0000 L CNN
 F 1 "220p" H 7640 2535 50  0000 L CNN
 F 2 "Capacitors_SMD:C_0402" H 7630 2615 50  0001 C CNN
@@
 $EndComp
 $Comp
-L C_Small C202
+L C_Small C201
 U 1 1 59D543D5
 P 7910 2605
-F 0 "C202" H 7920 2675 50  0000 L CNN
+F 0 "C201" H 7920 2675 50  0000 L CNN
 F 1 "220p" H 7920 2525 50  0000 L CNN
 F 2 "Capacitors_SMD:C_0402" H 7910 2605 50  0001 C CNN
@@
 $EndComp
 $Comp
-L GND #PWR212
+L GND #PWR213
 U 1 1 59D54491
 P 6490 3980
-F 0 "#PWR212" H 6490 3730 50  0001 C CNN
+F 0 "#PWR213" H 6490 3730 50  0001 C CNN
 F 1 "GND" H 6490 3830 50  0000 C CNN
 F 2 "" H 6490 3980 50  0001 C CNN
@@
 $EndComp
 $Comp
-L GND #PWR215
+L GND #PWR216
 U 1 1 5A9DC6DD
 P 4335 5065
-F 0 "#PWR215" H 4335 4815 50  0001 C CNN
+F 0 "#PWR216" H 4335 4815 50  0001 C CNN
 F 1 "GND" H 4335 4915 50  0000 C CNN
 F 2 "" H 4335 5065 50  0001 C CNN
@@
 $EndComp
 $Comp
-L GND #PWR213
+L GND #PWR214
 U 1 1 5A9DD534
 P 5075 4655
-F 0 "#PWR213" H 5075 4405 50  0001 C CNN
+F 0 "#PWR214" H 5075 4405 50  0001 C CNN
 F 1 "GND" H 5075 4505 50  0000 C CNN
 F 2 "" H 5075 4655 50  0001 C CNN
@@
 $EndComp
 $Comp
-L C_Small C201
+L C_Small C203
 U 1 1 5AB93975
 P 5725 2820
-F 0 "C201" H 5735 2890 50  0000 L CNN
+F 0 "C203" H 5735 2890 50  0000 L CNN
 F 1 "100n" H 5735 2740 50  0000 L CNN
 F 2 "Capacitors_SMD:C_0603_HandSoldering" H 5725 2820 50  0001 C CNN
@@
 $EndComp
 $Comp
-L GND #PWR214
+L GND #PWR215
 U 1 1 5AB97C20
 P 3080 4840
-F 0 "#PWR214" H 3080 4590 50  0001 C CNN
+F 0 "#PWR215" H 3080 4590 50  0001 C CNN
 F 1 "GND" H 3080 4690 50  0000 C CNN
 F 2 "" H 3080 4840 50  0001 C CNN
@@
 $EndComp
 $Comp
-L GND #PWR211
+L GND #PWR212
 U 1 1 5AB99878
 P 2605 3975
-F 0 "#PWR211" H 2605 3725 50  0001 C CNN
+F 0 "#PWR212" H 2605 3725 50  0001 C CNN
 F 1 "GND" H 2605 3825 50  0000 C CNN
 F 2 "" H 2605 3975 50  0001 C CNN
@@
 Wire Wire Line
 	6440 3820 6440 3910
-Connection ~ 7780 2795
 Wire Wire Line
 	7910 2795 7910 2705
@@
 	4135 4925 4135 5000
 Connection ~ 4235 5000
-Wire Wire Line
-	7785 2880 7785 2795
 Wire Wire Line
 	7340 2820 7430 2820
@@
 Wire Wire Line
 	1500 3680 1500 3605
+$Comp
+L GND #PWR211
+U 1 1 5AC9F292
+P 5440 3810
+F 0 "#PWR211" H 5440 3560 50  0001 C CNN
+F 1 "GND" H 5440 3660 50  0000 C CNN
+F 2 "" H 5440 3810 50  0001 C CNN
+F 3 "" H 5440 3810 50  0001 C CNN
+	1    5440 3810
+	1    0    0    -1
+$EndComp
+Wire Wire Line
+	5440 3810 5440 3725
+Connection ~ 5440 3725
+Wire Wire Line
+	7785 2880 7785 2795
+Connection ~ 7785 2795
 $EndSCHEMATC
