File: rf/rf2baseband.sch (KiCad schematic (older format))
At the start: 30 parts, among them U701 TLV4172

Commit message: Finish assigning component footprints
Parts:
- removed 100k: POT, symbol POT
- added RV601: 100k, rajsradar:RK09D113, symbol POT
- L607, L608: renamed from L?; footprint (none) -> Capacitors_SMD:C_0402
- R602, R603, R604, R607: renamed from R?; footprint (none) -> Resistors_SMD:R_0402
- gave numbers to parts that had none: 10
Connections:
- net at R604.1, U701.13 (-): now also RV601.1
- net at R603.2, U701.9 (-): now also RV601.3
- net at C606.1, U701.1: now also C609.2, R606.2; no longer C609.1, R606.1
- net at C608.2, U701.2 (-): now also R606.1; no longer R606.2
- net at C607.2, C608.1, R605.1: now also C609.1; no longer C609.2
Changed lines of the file:
@@
 $EndComp
 $Comp
-L +12V #PWR066
+L +12V #PWR603
 U 1 1 59E0B7DF
 P 5700 2705
-F 0 "#PWR066" H 5700 2555 50  0001 C CNN
+F 0 "#PWR603" H 5700 2555 50  0001 C CNN
 F 1 "+12V" H 5700 2845 50  0000 C CNN
 F 2 "" H 5700 2705 50  0001 C CNN
@@
 $EndComp
 $Comp
-L +12V #PWR067
+L +12V #PWR608
 U 1 1 59E0BA0D
 P 2485 4580
-F 0 "#PWR067" H 2485 4430 50  0001 C CNN
+F 0 "#PWR608" H 2485 4430 50  0001 C CNN
 F 1 "+12V" H 2485 4720 50  0000 C CNN
 F 2 "" H 2485 4580 50  0001 C CNN
@@
 $EndComp
 $Comp
-L GND #PWR068
+L GND #PWR615
 U 1 1 59E0BA54
 P 2485 5290
-F 0 "#PWR068" H 2485 5040 50  0001 C CNN
+F 0 "#PWR615" H 2485 5040 50  0001 C CNN
 F 1 "GND" H 2485 5140 50  0000 C CNN
 F 2 "" H 2485 5290 50  0001 C CNN
@@
 $EndComp
 $Comp
-L GND #PWR069
+L GND #PWR605
 U 1 1 59E0BA78
 P 5700 3625
-F 0 "#PWR069" H 5700 3375 50  0001 C CNN
+F 0 "#PWR605" H 5700 3375 50  0001 C CNN
 F 1 "GND" H 5700 3475 50  0000 C CNN
 F 2 "" H 5700 3625 50  0001 C CNN
@@
 $EndComp
 $Comp
-L +6V #PWR070
+L +6V #PWR609
 U 1 1 59E0BD90
 P 2740 4735
-F 0 "#PWR070" H 2740 4585 50  0001 C CNN
+F 0 "#PWR609" H 2740 4585 50  0001 C CNN
 F 1 "+6V" H 2740 4875 50  0000 C CNN
 F 2 "" H 2740 4735 50  0001 C CNN
@@
 100kHz LPF
 $Comp
-L +12V #PWR073
+L +12V #PWR610
 U 1 1 59E1133D
 P 1625 4775
-F 0 "#PWR073" H 1625 4625 50  0001 C CNN
+F 0 "#PWR610" H 1625 4625 50  0001 C CNN
 F 1 "+12V" H 1625 4915 50  0000 C CNN
 F 2 "" H 1625 4775 50  0001 C CNN
@@
 $EndComp
 $Comp
-L +12VA #PWR074
+L +12VA #PWR607
 U 1 1 59E119E6
 P 995 4475
-F 0 "#PWR074" H 995 4325 50  0001 C CNN
+F 0 "#PWR607" H 995 4325 50  0001 C CNN
 F 1 "+12VA" H 995 4615 50  0000 C CNN
 F 2 "" H 995 4475 50  0001 C CNN
@@
 $EndComp
 $Comp
-L GND #PWR075
+L GND #PWR611
 U 1 1 59E1200C
 P 995 5135
-F 0 "#PWR075" H 995 4885 50  0001 C CNN
+F 0 "#PWR611" H 995 4885 50  0001 C CNN
 F 1 "GND" H 995 4985 50  0000 C CNN
 F 2 "" H 995 5135 50  0001 C CNN
@@
 $EndComp
 $Comp
-L GND #PWR076
+L GND #PWR612
 U 1 1 59E12063
 P 1205 5135
-F 0 "#PWR076" H 1205 4885 50  0001 C CNN
+F 0 "#PWR612" H 1205 4885 50  0001 C CNN
 F 1 "GND" H 1205 4985 50  0000 C CNN
 F 2 "" H 1205 5135 50  0001 C CNN
@@
 $EndComp
 $Comp
-L GND #PWR077
+L GND #PWR613
 U 1 1 59E120B3
 P 1425 5135
-F 0 "#PWR077" H 1425 4885 50  0001 C CNN
+F 0 "#PWR613" H 1425 4885 50  0001 C CNN
 F 1 "GND" H 1425 4985 50  0000 C CNN
 F 2 "" H 1425 5135 50  0001 C CNN
@@
 $EndComp
 $Comp
-L GND #PWR078
+L GND #PWR614
 U 1 1 59E12103
 P 1625 5135
-F 0 "#PWR078" H 1625 4885 50  0001 C CNN
+F 0 "#PWR614" H 1625 4885 50  0001 C CNN
 F 1 "GND" H 1625 4985 50  0000 C CNN
 F 2 "" H 1625 5135 50  0001 C CNN
@@
 $EndComp
 $Comp
-L L_Small L?
+L L_Small L607
 U 1 1 5ABD47F6
 P 2425 2525
-F 0 "L?" H 2455 2565 50  0000 L CNN
+F 0 "L607" H 2455 2565 50  0000 L CNN
 F 1 "1uH" H 2455 2485 50  0000 L CNN
-F 2 "" H 2425 2525 50  0001 C CNN
+F 2 "Capacitors_SMD:C_0402" H 2425 2525 50  0001 C CNN
 F 3 "" H 2425 2525 50  0001 C CNN
 	1    2425 2525
@@
 $EndComp
 $Comp
-L L_Small L?
+L L_Small L608
 U 1 1 5ABE83C5
 P 2425 2850
-F 0 "L?" H 2455 2890 50  0000 L CNN
+F 0 "L608" H 2455 2890 50  0000 L CNN
 F 1 "1uH" H 2455 2810 50  0000 L CNN
-F 2 "" H 2425 2850 50  0001 C CNN
+F 2 "Capacitors_SMD:C_0402" H 2425 2850 50  0001 C CNN
 F 3 "" H 2425 2850 50  0001 C CNN
 	1    2425 2850
@@
 $EndComp
 $Comp
-L R_Small R?
+L R_Small R601
 U 1 1 5ABEFACC
 P 5055 1790
-F 0 "R?" H 5085 1810 50  0000 L CNN
+F 0 "R601" H 5085 1810 50  0000 L CNN
 F 1 "1k" H 5085 1750 50  0000 L CNN
 F 2 "Resistors_SMD:R_1206_HandSoldering" H 5055 1790 50  0001 C CNN
@@
 $EndComp
 $Comp
-L C_Small C?
+L C_Small C605
 U 1 1 5ABEFBA2
 P 4840 2035
-F 0 "C?" H 4850 2105 50  0000 L CNN
+F 0 "C605" H 4850 2105 50  0000 L CNN
 F 1 "8n5" H 4850 1955 50  0000 L CNN
 F 2 "Capacitors_SMD:C_0603_HandSoldering" H 4840 2035 50  0001 C CNN
@@
 $EndComp
 $Comp
-L C_Small C?
+L C_Small C610
 U 1 1 5ABF9B08
 P 2740 5280
-F 0 "C?" H 2750 5350 50  0000 L CNN
+F 0 "C610" H 2750 5350 50  0000 L CNN
 F 1 "100n" H 2750 5200 50  0000 L CNN
 F 2 "Capacitors_SMD:C_0603_HandSoldering" H 2740 5280 50  0001 C CNN
@@
 $EndComp
 $Comp
-L C_Small C?
+L C_Small C611
 U 1 1 5ABF9BC7
 P 2990 5280
-F 0 "C?" H 3000 5350 50  0000 L CNN
+F 0 "C611" H 3000 5350 50  0000 L CNN
 F 1 "1u" H 3000 5200 50  0000 L CNN
 F 2 "Capacitors_SMD:C_0603_HandSoldering" H 2990 5280 50  0001 C CNN
@@
 $EndComp
 $Comp
-L GND #PWR?
+L GND #PWR616
 U 1 1 5ABF9C45
 P 2990 5535
-F 0 "#PWR?" H 2990 5285 50  0001 C CNN
+F 0 "#PWR616" H 2990 5285 50  0001 C CNN
 F 1 "GND" H 2990 5385 50  0000 C CNN
 F 2 "" H 2990 5535 50  0001 C CNN
@@
 $EndComp
 $Comp
-L R_Small R?
+L R_Small R604
 U 1 1 5AC25582
 P 3590 2945
-F 0 "R?" H 3620 2965 50  0000 L CNN
+F 0 "R604" H 3620 2965 50  0000 L CNN
 F 1 "100k" H 3620 2905 50  0000 L CNN
-F 2 "" H 3590 2945 50  0001 C CNN
+F 2 "Resistors_SMD:R_0402" H 3590 2945 50  0001 C CNN
 F 3 "" H 3590 2945 50  0001 C CNN
 	1    3590 2945
@@
 $EndComp
 $Comp
-L R_Small R?
+L R_Small R603
 U 1 1 5AC256A2
 P 3550 2435
-F 0 "R?" H 3580 2455 50  0000 L CNN
+F 0 "R603" H 3580 2455 50  0000 L CNN
 F 1 "100k" H 3580 2395 50  0000 L CNN
-F 2 "" H 3550 2435 50  0001 C CNN
+F 2 "Resistors_SMD:R_0402" H 3550 2435 50  0001 C CNN
 F 3 "" H 3550 2435 50  0001 C CNN
 	1    3550 2435
@@
 $EndComp
 $Comp
-L POT 100k
-U 1 1 5AC25BB4
-P 3120 2715
-F 0 "100k" V 2945 2715 50  0000 C CNN
-F 1 "POT" V 3020 2715 50  0000 C CNN
-F 2 "" H 3120 2715 50  0001 C CNN
-F 3 "" H 3120 2715 50  0001 C CNN
-	1    3120 2715
-	-1   0    0    1
-$EndComp
-$Comp
-L R_Small R?
+L R_Small R605
 U 1 1 5AC2C319
 P 4820 2990
-F 0 "R?" H 4850 3010 50  0000 L CNN
+F 0 "R605" H 4850 3010 50  0000 L CNN
 F 1 "165" H 4850 2950 50  0000 L CNN
 F 2 "Resistors_SMD:R_1206_HandSoldering" H 4820 2990 50  0001 C CNN
@@
 $EndComp
 $Comp
-L C_Small C?
+L C_Small C607
 U 1 1 5AC2C31F
 P 4530 3295
-F 0 "C?" H 4540 3365 50  0000 L CNN
+F 0 "C607" H 4540 3365 50  0000 L CNN
 F 1 "8n5" H 4540 3215 50  0000 L CNN
 F 2 "Capacitors_SMD:C_0603_HandSoldering" H 4530 3295 50  0001 C CNN
@@
 $EndComp
 $Comp
-L C_Small C?
+L C_Small C609
 U 1 1 5AC2C325
 P 4670 3570
-F 0 "C?" H 4680 3640 50  0000 L CNN
+F 0 "C609" H 4680 3640 50  0000 L CNN
 F 1 "2n2" H 4680 3490 50  0000 L CNN
 F 2 "Capacitors_SMD:C_0603_HandSoldering" H 4670 3570 50  0001 C CNN
 F 3 "" H 4670 3570 50  0001 C CNN
 	1    4670 3570
-	1    0    0    1
-$EndComp
-$Comp
-L C_Small C?
+	1    0    0    -1
+$EndComp
+$Comp
+L C_Small C606
 U 1 1 5AC2C32B
 P 6470 3195
-F 0 "C?" H 6480 3265 50  0000 L CNN
+F 0 "C606" H 6480 3265 50  0000 L CNN
 F 1 "1u" H 6480 3115 50  0000 L CNN
 F 2 "Capacitors_SMD:C_0603_HandSoldering" H 6470 3195 50  0001 C CNN
@@
 $EndComp
 $Comp
-L R_Small R?
+L R_Small R606
 U 1 1 5AC2C337
 P 5260 3540
-F 0 "R?" H 5290 3560 50  0000 L CNN
+F 0 "R606" H 5290 3560 50  0000 L CNN
 F 1 "1k" H 5290 3500 50  0000 L CNN
 F 2 "Resistors_SMD:R_1206_HandSoldering" H 5260 3540 50  0001 C CNN
 F 3 "" H 5260 3540 50  0001 C CNN
 	1    5260 3540
-	1    0    0    1
-$EndComp
-$Comp
-L C_Small C?
+	1    0    0    -1
+$EndComp
+$Comp
+L C_Small C608
 U 1 1 5AC2C33D
 P 5045 3295
-F 0 "C?" H 5055 3365 50  0000 L CNN
+F 0 "C608" H 5055 3365 50  0000 L CNN
 F 1 "8n5" H 5055 3215 50  0000 L CNN
 F 2 "Capacitors_SMD:C_0603_HandSoldering" H 5045 3295 50  0001 C CNN
@@
 $EndComp
 $Comp
-L +6V #PWR?
+L +6V #PWR602
 U 1 1 5ABF1671
 P 5275 2510
-F 0 "#PWR?" H 5275 2360 50  0001 C CNN
+F 0 "#PWR602" H 5275 2360 50  0001 C CNN
 F 1 "+6V" H 5275 2650 50  0000 C CNN
 F 2 "" H 5275 2510 50  0001 C CNN
@@
 $EndComp
 $Comp
-L GND #PWR?
+L GND #PWR604
 U 1 1 5AC2FDF8
 P 4445 2725
-F 0 "#PWR?" H 4445 2475 50  0001 C CNN
+F 0 "#PWR604" H 4445 2475 50  0001 C CNN
 F 1 "GND" H 4445 2575 50  0000 C CNN
 F 2 "" H 4445 2725 50  0001 C CNN
@@
 OUT-
 $Comp
-L R_Small R?
+L R_Small R607
 U 1 1 5AC322CC
 P 2650 3550
-F 0 "R?" H 2680 3570 50  0000 L CNN
+F 0 "R607" H 2680 3570 50  0000 L CNN
 F 1 "100k" H 2680 3510 50  0000 L CNN
-F 2 "" H 2650 3550 50  0001 C CNN
+F 2 "Resistors_SMD:R_0402" H 2650 3550 50  0001 C CNN
 F 3 "" H 2650 3550 50  0001 C CNN
 	1    2650 3550
@@
 $EndComp
 $Comp
-L R_Small R?
+L R_Small R602
 U 1 1 5AC32DCD
 P 2650 1845
-F 0 "R?" H 2680 1865 50  0000 L CNN
+F 0 "R602" H 2680 1865 50  0000 L CNN
 F 1 "100k" H 2680 1805 50  0000 L CNN
-F 2 "" H 2650 1845 50  0001 C CNN
+F 2 "Resistors_SMD:R_0402" H 2650 1845 50  0001 C CNN
 F 3 "" H 2650 1845 50  0001 C CNN
 	1    2650 1845
@@
 Connection ~ 2650 2025
 $Comp
-L +6V #PWR?
+L +6V #PWR601
 U 1 1 5AC34C21
 P 2650 1660
-F 0 "#PWR?" H 2650 1510 50  0001 C CNN
+F 0 "#PWR601" H 2650 1510 50  0001 C CNN
 F 1 "+6V" H 2650 1800 50  0000 C CNN
 F 2 "" H 2650 1660 50  0001 C CNN
@@
 	2650 1660 2650 1745
 $Comp
-L +6V #PWR?
+L +6V #PWR606
 U 1 1 5AC34E47
 P 2650 3730
-F 0 "#PWR?" H 2650 3580 50  0001 C CNN
+F 0 "#PWR606" H 2650 3580 50  0001 C CNN
 F 1 "+6V" H 2650 3870 50  0000 C CNN
 F 2 "" H 2650 3730 50  0001 C CNN
@@
 	-1   0    0    1
 $EndComp
+$Comp
+L POT RV601
+U 1 1 5AC6CA82
+P 3120 2715
+F 0 "RV601" V 2945 2715 50  0000 C CNN
+F 1 "100k" V 3020 2715 50  0000 C CNN
+F 2 "rajsradar:RK09D113" H 3120 2715 50  0001 C CNN
+F 3 "" H 3120 2715 50  0001 C CNN
+	1    3120 2715
+	-1   0    0    1
+$EndComp

Commit message: Finish first revision layout
Parts:
- renumbered C701 to C601, C704 to C602, C605 to C603, C702 to C604, C703 to C605, C705 to C610, C706 to C611, C707 to C612, C708 to C613, C610 to C614, C611 to C615, L607 to L601, L608 to L602, L701 to L603, R704 to R603, R603 to R604, R604 to R605, R605 to R606, R606 to R607, R607 to R608, R708 to R609, R709 to R610, U701 to U601
Connections:
- net +12V: now also U601.11; no longer U601.11
- net +6V: now also U601.3 (+); no longer U601.3 (+)
- net GND: now also U601.4; no longer U601.4
- net at C605.2, L601.2, R602.2: now also U601.10 (+); no longer U601.10 (+)
- net at C602.1, R604.1: now also U601.8; no longer U601.8
- net at R604.2, RV601.3: now also RV601.2, U601.9 (-); no longer U601.9 (-)
- net at C606.1, C609.2, R607.2: now also U601.1; no longer U601.1
- net at C608.2, R607.1: now also U601.2 (-); no longer U601.2 (-)
Changed lines of the file:
@@
 LIBS:mc2016k30
 LIBS:cp0402q5425entr
+LIBS:lm340-5
 EELAYER 25 0
 EELAYER END
@@
 $EndDescr
 $Comp
-L TLV4172 U701
+L TLV4172 U601
 U 4 1 59DEF024
 P 3620 3285
-F 0 "U701" H 3620 3285 60  0000 C CNN
+F 0 "U601" H 3620 3285 60  0000 C CNN
 F 1 "TLV4172" H 3820 3135 60  0000 C CNN
 F 2 "Housings_SSOP:TSSOP-14_4.4x5mm_Pitch0.65mm" H 3620 3285 60  0001 C CNN
@@
 $EndComp
 $Comp
-L TLV4172 U701
-U 3 1 59DEF055
+L TLV4172 U601
+U 1 1 59DEF055
+P 5800 3195
+F 0 "U601" H 5800 3195 60  0000 C CNN
+F 1 "TLV4172" H 6000 3045 60  0000 C CNN
+F 2 "Housings_SSOP:TSSOP-14_4.4x5mm_Pitch0.65mm" H 5800 3195 60  0001 C CNN
+F 3 "" H 5800 3195 60  0001 C CNN
+	1    5800 3195
+	1    0    0    1
+$EndComp
+$Comp
+L TLV4172 U601
+U 2 1 59DEF098
+P 5595 2135
+F 0 "U601" H 5595 2135 60  0000 C CNN
+F 1 "TLV4172" H 5795 1985 60  0000 C CNN
+F 2 "Housings_SSOP:TSSOP-14_4.4x5mm_Pitch0.65mm" H 5595 2135 60  0001 C CNN
+F 3 "" H 5595 2135 60  0001 C CNN
+	2    5595 2135
+	1    0    0    -1
+$EndComp
+$Comp
+L TLV4172 U601
+U 3 1 59DEF0E7
 P 3680 2125
-F 0 "U701" H 3680 2125 60  0000 C CNN
+F 0 "U601" H 3680 2125 60  0000 C CNN
 F 1 "TLV4172" H 3880 1975 60  0000 C CNN
 F 2 "Housings_SSOP:TSSOP-14_4.4x5mm_Pitch0.65mm" H 3680 2125 60  0001 C CNN
 F 3 "" H 3680 2125 60  0001 C CNN
 	3    3680 2125
-	1    0    0    1
-$EndComp
-$Comp
-L TLV4172 U701
-U 2 1 59DEF098
-P 5595 2135
-F 0 "U701" H 5595 2135 60  0000 C CNN
-F 1 "TLV4172" H 5795 1985 60  0000 C CNN
-F 2 "Housings_SSOP:TSSOP-14_4.4x5mm_Pitch0.65mm" H 5595 2135 60  0001 C CNN
-F 3 "" H 5595 2135 60  0001 C CNN
-	2    5595 2135
-	1    0    0    -1
-$EndComp
-$Comp
-L TLV4172 U701
-U 1 1 59DEF0E7
-P 5800 3195
-F 0 "U701" H 5800 3195 60  0000 C CNN
-F 1 "TLV4172" H 6000 3045 60  0000 C CNN
-F 2 "Housings_SSOP:TSSOP-14_4.4x5mm_Pitch0.65mm" H 5800 3195 60  0001 C CNN
-F 3 "" H 5800 3195 60  0001 C CNN
-	1    5800 3195
 	1    0    0    1
 $EndComp
@@
 $EndComp
 $Comp
-L R_Small R708
+L R_Small R609
 U 1 1 59E0B935
 P 2485 4770
-F 0 "R708" H 2515 4790 50  0000 L CNN
+F 0 "R609" H 2515 4790 50  0000 L CNN
 F 1 "10k" H 2515 4730 50  0000 L CNN
 F 2 "Resistors_SMD:R_0402" H 2485 4770 50  0001 C CNN
@@
 $EndComp
 $Comp
-L R_Small R709
+L R_Small R610
 U 1 1 59E0B9CB
 P 2485 5110
-F 0 "R709" H 2515 5130 50  0000 L CNN
+F 0 "R610" H 2515 5130 50  0000 L CNN
 F 1 "10k" H 2515 5070 50  0000 L CNN
 F 2 "Resistors_SMD:R_0402" H 2485 5110 50  0001 C CNN
@@
 INM
 $Comp
-L C_Small C703
+L C_Small C605
 U 1 1 59E0CB5D
 P 2650 2700
-F 0 "C703" H 2660 2770 50  0000 L CNN
+F 0 "C605" H 2660 2770 50  0000 L CNN
 F 1 "5n6" H 2660 2620 50  0000 L CNN
 F 2 "Capacitors_SMD:C_0603_HandSoldering" H 2650 2700 50  0001 C CNN
@@
 $EndComp
 $Comp
-L R_Small R704
+L R_Small R603
 U 1 1 59E0E10A
 P 4615 2340
-F 0 "R704" H 4645 2360 50  0000 L CNN
+F 0 "R603" H 4645 2360 50  0000 L CNN
 F 1 "165" H 4645 2300 50  0000 L CNN
 F 2 "Resistors_SMD:R_1206_HandSoldering" H 4615 2340 50  0001 C CNN
@@
 $EndComp
 $Comp
-L C_Small C704
+L C_Small C602
 U 1 1 59E0E1D3
 P 4325 2035
-F 0 "C704" H 4335 2105 50  0000 L CNN
+F 0 "C602" H 4335 2105 50  0000 L CNN
 F 1 "8n5" H 4335 1955 50  0000 L CNN
 F 2 "Capacitors_SMD:C_0603_HandSoldering" H 4325 2035 50  0001 C CNN
@@
 $EndComp
 $Comp
-L C_Small C701
+L C_Small C601
 U 1 1 59E0E272
 P 4465 1760
-F 0 "C701" H 4475 1830 50  0000 L CNN
+F 0 "C601" H 4475 1830 50  0000 L CNN
 F 1 "2n2" H 4475 1680 50  0000 L CNN
 F 2 "Capacitors_SMD:C_0603_HandSoldering" H 4465 1760 50  0001 C CNN
@@
 $EndComp
 $Comp
-L C_Small C702
+L C_Small C604
 U 1 1 59E0E7CF
 P 6265 2135
-F 0 "C702" H 6275 2205 50  0000 L CNN
+F 0 "C604" H 6275 2205 50  0000 L CNN
 F 1 "1u" H 6275 2055 50  0000 L CNN
 F 2 "Capacitors_SMD:C_0603_HandSoldering" H 6265 2135 50  0001 C CNN
@@
 $EndComp
 $Comp
-L C_Small C706
+L C_Small C611
 U 1 1 59E11387
 P 1205 4975
-F 0 "C706" H 1215 5045 50  0000 L CNN
+F 0 "C611" H 1215 5045 50  0000 L CNN
 F 1 "10u" H 1215 4895 50  0000 L CNN
 F 2 "Capacitors_SMD:C_0805_HandSoldering" H 1205 4975 50  0001 C CNN
@@
 $EndComp
 $Comp
-L C_Small C705
+L C_Small C610
 U 1 1 59E1149D
 P 995 4975
-F 0 "C705" H 1005 5045 50  0000 L CNN
+F 0 "C610" H 1005 5045 50  0000 L CNN
 F 1 "22u" H 1005 4895 50  0000 L CNN
 F 2 "Capacitors_SMD:C_1210_HandSoldering" H 995 4975 50  0001 C CNN
@@
 $EndComp
 $Comp
-L C_Small C707
+L C_Small C612
 U 1 1 59E11519
 P 1425 4975
-F 0 "C707" H 1435 5045 50  0000 L CNN
+F 0 "C612" H 1435 5045 50  0000 L CNN
 F 1 "1u" H 1435 4895 50  0000 L CNN
 F 2 "Capacitors_SMD:C_0603_HandSoldering" H 1425 4975 50  0001 C CNN
@@
 $EndComp
 $Comp
-L C_Small C708
+L C_Small C613
 U 1 1 59E1158A
 P 1625 4975
-F 0 "C708" H 1635 5045 50  0000 L CNN
+F 0 "C613" H 1635 5045 50  0000 L CNN
 F 1 "100n" H 1635 4895 50  0000 L CNN
 F 2 "Capacitors_SMD:C_0603_HandSoldering" H 1625 4975 50  0001 C CNN
@@
 $EndComp
 $Comp
-L L_Core_Ferrite_Small L701
+L L_Core_Ferrite_Small L603
 U 1 1 59E16A96
 P 995 4665
-F 0 "L701" H 1045 4705 50  0000 L CNN
+F 0 "L603" H 1045 4705 50  0000 L CNN
 F 1 "1k@190MHz" H 1045 4615 50  0000 L CNN
 F 2 "Capacitors_SMD:C_0402" H 995 4665 50  0001 C CNN
@@
 $EndComp
 $Comp
-L L_Small L607
+L L_Small L601
 U 1 1 5ABD47F6
 P 2425 2525
-F 0 "L607" H 2455 2565 50  0000 L CNN
+F 0 "L601" H 2455 2565 50  0000 L CNN
 F 1 "1uH" H 2455 2485 50  0000 L CNN
 F 2 "Capacitors_SMD:C_0402" H 2425 2525 50  0001 C CNN
@@
 $EndComp
 $Comp
-L L_Small L608
+L L_Small L602
 U 1 1 5ABE83C5
 P 2425 2850
-F 0 "L608" H 2455 2890 50  0000 L CNN
+F 0 "L602" H 2455 2890 50  0000 L CNN
 F 1 "1uH" H 2455 2810 50  0000 L CNN
 F 2 "Capacitors_SMD:C_0402" H 2425 2850 50  0001 C CNN
@@
 $EndComp
 $Comp
-L C_Small C605
+L C_Small C603
 U 1 1 5ABEFBA2
 P 4840 2035
-F 0 "C605" H 4850 2105 50  0000 L CNN
+F 0 "C603" H 4850 2105 50  0000 L CNN
 F 1 "8n5" H 4850 1955 50  0000 L CNN
 F 2 "Capacitors_SMD:C_0603_HandSoldering" H 4840 2035 50  0001 C CNN
@@
 $EndComp
 $Comp
-L C_Small C610
+L C_Small C614
 U 1 1 5ABF9B08
 P 2740 5280
-F 0 "C610" H 2750 5350 50  0000 L CNN
+F 0 "C614" H 2750 5350 50  0000 L CNN
 F 1 "100n" H 2750 5200 50  0000 L CNN
 F 2 "Capacitors_SMD:C_0603_HandSoldering" H 2740 5280 50  0001 C CNN
@@
 $EndComp
 $Comp
-L C_Small C611
+L C_Small C615
 U 1 1 5ABF9BC7
 P 2990 5280
-F 0 "C611" H 3000 5350 50  0000 L CNN
+F 0 "C615" H 3000 5350 50  0000 L CNN
 F 1 "1u" H 3000 5200 50  0000 L CNN
 F 2 "Capacitors_SMD:C_0603_HandSoldering" H 2990 5280 50  0001 C CNN
@@
 $EndComp
 $Comp
-L R_Small R604
+L R_Small R605
 U 1 1 5AC25582
 P 3590 2945
-F 0 "R604" H 3620 2965 50  0000 L CNN
+F 0 "R605" H 3620 2965 50  0000 L CNN
 F 1 "100k" H 3620 2905 50  0000 L CNN
 F 2 "Resistors_SMD:R_0402" H 3590 2945 50  0001 C CNN
@@
 $EndComp
 $Comp
-L R_Small R603
+L R_Small R604
 U 1 1 5AC256A2
 P 3550 2435
-F 0 "R603" H 3580 2455 50  0000 L CNN
+F 0 "R604" H 3580 2455 50  0000 L CNN
 F 1 "100k" H 3580 2395 50  0000 L CNN
 F 2 "Resistors_SMD:R_0402" H 3550 2435 50  0001 C CNN
@@
 $EndComp
 $Comp
-L R_Small R605
+L R_Small R606
 U 1 1 5AC2C319
 P 4820 2990
-F 0 "R605" H 4850 3010 50  0000 L CNN
+F 0 "R606" H 4850 3010 50  0000 L CNN
 F 1 "165" H 4850 2950 50  0000 L CNN
 F 2 "Resistors_SMD:R_1206_HandSoldering" H 4820 2990 50  0001 C CNN
@@
 $EndComp
 $Comp
-L R_Small R606
+L R_Small R607
 U 1 1 5AC2C337
 P 5260 3540
-F 0 "R606" H 5290 3560 50  0000 L CNN
+F 0 "R607" H 5290 3560 50  0000 L CNN
 F 1 "1k" H 5290 3500 50  0000 L CNN
 F 2 "Resistors_SMD:R_1206_HandSoldering" H 5260 3540 50  0001 C CNN
@@
 OUT-
 $Comp
-L R_Small R607
+L R_Small R608
 U 1 1 5AC322CC
 P 2650 3550
-F 0 "R607" H 2680 3570 50  0000 L CNN
+F 0 "R608" H 2680 3570 50  0000 L CNN
 F 1 "100k" H 2680 3510 50  0000 L CNN
 F 2 "Resistors_SMD:R_0402" H 2650 3550 50  0001 C CNN
@@
 Wire Wire Line
 	2970 2715 2910 2715
-Connection ~ 3120 2495
 Wire Wire Line
 	3690 2945 4050 2945
@@
 Connection ~ 2650 2850
 Wire Wire Line
-	3120 2500 2910 2500
-Wire Wire Line
-	2910 2500 2910 2715
+	2910 2715 2910 2500
 Wire Wire Line
 	4130 2035 4130 2435
@@
 	-1   0    0    1
 $EndComp
+Wire Wire Line
+	2910 2500 3120 2500
+Connection ~ 3120 2500
 $EndSCHEMATC
