File: digital/digital.sch (KiCad schematic (older format))
At the start: 46 parts, among them J101 BASEBAND, J102 LNA_INTERFACE, J103 VCO_INTERFACE, J104 RF_POWER, J105 UART, J106 PLL_INTERFACE, J107 PA_INTERFACE, J108 USB_OTG, J109 FPGA_PROG, J110 SWD/JTAG, J111 PWR_IN, Q101 Q_PMOS_GSD, U101 LDK320AM33R, U102 TPS54308

Commit message: Finish digital layout
Parts:
- TP101, TP102, TP103, TP104, TP105: footprint SMD_Packages:1Pin -> Measurement_Points:Measurement_Point_Round-SMD-Pad_Small
Connections:
- net FLASH_CSN: now also J109.3 (Pin_3); no longer J109.5 (Pin_5)
- net FLASH_MISO: now also J109.4 (Pin_4); no longer J109.3 (Pin_3)
- net FLASH_MOSI: now also J109.5 (Pin_5); no longer J109.4 (Pin_4)
- net FLASH_SCK: now also J109.6 (Pin_6); no longer J109.2 (Pin_2)
- net FPGA_RSTN: now also J109.7 (Pin_7); no longer J109.6 (Pin_6)
Changed lines of the file:
@@
 LIBS:tlv74125pdbvr
 LIBS:opa2376qdgkrq1
+LIBS:tlv74312pdbvr
 LIBS:digital-cache
 EELAYER 25 0
@@
 F 0 "TP101" H 5550 1250 50  0000 C BNN
 F 1 "TEST" H 5550 1200 50  0000 C CNN
-F 2 "SMD_Packages:1Pin" H 5550 950 50  0001 C CNN
+F 2 "Measurement_Points:Measurement_Point_Round-SMD-Pad_Small" H 5550 950 50  0001 C CNN
 F 3 "" H 5550 950 50  0001 C CNN
 	1    5550 950
@@
 F 0 "TP102" H 5600 1350 50  0000 C BNN
 F 1 "TEST" H 5600 1300 50  0000 C CNN
-F 2 "SMD_Packages:1Pin" H 5600 1050 50  0001 C CNN
+F 2 "Measurement_Points:Measurement_Point_Round-SMD-Pad_Small" H 5600 1050 50  0001 C CNN
 F 3 "" H 5600 1050 50  0001 C CNN
 	1    5600 1050
@@
 Text Label 2200 6350 0    60   ~ 0
 USB_D-
-Text Label 1000 6150 0    60   ~ 0
+Text Label 1000 6550 0    60   ~ 0
 FLASH_SCK
+Text Label 1000 6350 0    60   ~ 0
+FLASH_MISO
+Text Label 1000 6450 0    60   ~ 0
+FLASH_MOSI
 Text Label 1000 6250 0    60   ~ 0
-FLASH_MISO
-Text Label 1000 6350 0    60   ~ 0
-FLASH_MOSI
-Text Label 1000 6450 0    60   ~ 0
 FLASH_CSN
-Text Label 1000 6550 0    60   ~ 0
+Text Label 1000 6650 0    60   ~ 0
 FPGA_RSTN
 Text Label 5550 6550 2    60   ~ 0
@@
 F 0 "TP103" H 8150 1400 50  0000 C BNN
 F 1 "TEST" H 8150 1350 50  0000 C CNN
-F 2 "SMD_Packages:1Pin" H 8150 1100 50  0001 C CNN
+F 2 "Measurement_Points:Measurement_Point_Round-SMD-Pad_Small" H 8150 1100 50  0001 C CNN
 F 3 "" H 8150 1100 50  0001 C CNN
 	1    8150 1100
@@
 F 0 "TP105" H 8250 1500 50  0000 C BNN
 F 1 "TEST" H 8250 1450 50  0000 C CNN
-F 2 "SMD_Packages:1Pin" H 8250 1200 50  0001 C CNN
+F 2 "Measurement_Points:Measurement_Point_Round-SMD-Pad_Small" H 8250 1200 50  0001 C CNN
 F 3 "" H 8250 1200 50  0001 C CNN
 	1    8250 1200
@@
 F 0 "TP104" H 8350 1400 50  0000 C BNN
 F 1 "TEST" H 8350 1350 50  0000 C CNN
-F 2 "SMD_Packages:1Pin" H 8350 1100 50  0001 C CNN
+F 2 "Measurement_Points:Measurement_Point_Round-SMD-Pad_Small" H 8350 1100 50  0001 C CNN
 F 3 "" H 8350 1100 50  0001 C CNN
 	1    8350 1100
@@
 	5050 2450 5850 2450
 Wire Wire Line
-	1000 6150 1550 6150
-Wire Wire Line
 	5050 2350 5850 2350
 Wire Wire Line
@@
 $EndComp
 NoConn ~ 6400 4300
-NoConn ~ 1550 6650
 $Comp
 L C_Small C107
@@
 	4150 3800 4150 3900
 Connection ~ 4000 3800
+Wire Wire Line
+	1000 6650 1550 6650
+NoConn ~ 1550 6150
 $EndSCHEMATC
