File: digital/ice40.sch (KiCad schematic (older format))
At the start: 31 parts

Commit message: Finish schematic TODO footprints
Parts:
- added C319: 10u, symbol C_Small
- added C320: 100n, symbol C_Small
- added U304: TLV74125PDBVR, symbol TLV74125PDBVR
- C310: renamed from C?; value 0u1 -> 100n
- gave numbers to parts that had none: 27
Connections:
- net labels added: +3.3V
- net labels removed: +2V5
- wire segments 125 -> 134
Other:
- moved on the sheet: C301, C302, C303, C304, C305, C306, C307, C308, C309, C311, C312, C313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

Commit message: Finish schematic and footprinting of digital board
Parts:
- added R308: 10k, Resistors_SMD:R_0603_HandSoldering, symbol R_Small
- C301, C303, C304, C307, C309, C312, C313, C315, C317, C319: footprint (none) -> Capacitors_SMD:C_0805_HandSoldering
- C302, C305, C306, C308, C310, C311, C314, C316, C318, C320: footprint (none) -> Capacitors_SMD:C_0603_HandSoldering
- R301: value 5k -> 10k; footprint (none) -> Resistors_SMD:R_0603_HandSoldering
- R302, R304, R305, R306, R307: footprint (none) -> Resistors_SMD:R_0603_HandSoldering
- R303: footprint (none) -> Resistors_SMD:R_0402
- U301: footprint (none) -> digital:Lattice_QFN48
- U302: footprint (none) -> Crystals:Crystal_SMD_3225-4pin_3.2x2.5mm_HandSoldering
- U303: footprint (none) -> Housings_SOIC:SOIC-8_3.9x4.9mm_Pitch1.27mm
- U304: footprint (none) -> TO_SOT_Packages_SMD:SOT-23-5_HandSoldering
Connections:
- net +3V3: now also R308.1
- net CDONE: now also R308.2
- no-connect marks 1 -> 22

Commit message: Finish digital layout
Parts:
- removed C303: 10u, Capacitors_SMD:C_0805_HandSoldering, symbol C_Small
- added C321: 100n, Capacitors_SMD:C_0603_HandSoldering, symbol C_Small
- added C322: 10u, Capacitors_SMD:C_0805_HandSoldering, symbol C_Small
- added U305: TLV74312PDBVR, TO_SOT_Packages_SMD:SOT-23-5_HandSoldering, symbol TLV74312PDBVR
Connections:
- net +1V2: now also U305.5 (OUT)
- net +3V3: now also C321.1, C322.1, U305.1 (IN), U305.3 (EN)
- net GND: now also C321.2, C322.2, U305.2 (GND)
- net PLL_CLK: now also U301.28 (IOT_41a); no longer U301.25 (IOT_36b)
- net PLL_DATA: now also U301.27 (IOT_38b); no longer U301.26 (IOT_39a)
- net PLL_LE: now also U301.26 (IOT_39a); no longer U301.27 (IOT_38b)
- net PLL_MUXOUT: now also U301.4 (IOB_8a); no longer U301.28 (IOT_41a)
- net SPI0_CLK: now also U301.11 (IOB_20a); no longer U301.46 (IOB_0a)
- net SPI0_CSN: now also U301.12 (IOB_22a); no longer U301.48 (IOB_4a)
- net SPI0_MISO: now also U301.10 (IOB_18a); no longer U301.47 (IOB_2a)
- net SPI0_MOSI: now also U301.9 (IOB_16a); no longer U301.45 (IOB_5b)
- net SPI1_MISO: now also U301.20 (IOB_25b_G3); no longer U301.19 (IOB_29b)
- net SPI1_SCK: now also U301.19 (IOB_29b); no longer U301.20 (IOB_25b_G3)
Changed lines of the file:
@@
 LIBS:tlv74125pdbvr
 LIBS:opa2376qdgkrq1
+LIBS:tlv74312pdbvr
 LIBS:digital-cache
 EELAYER 25 0
@@
 $Comp
 L ICE5LP1K-SG48ITR50 U301
-U 1 1 5AD1908F
-P 4150 2000
-F 0 "U301" H 4150 2000 60  0000 C CNN
-F 1 "ICE5LP1K-SG48ITR50" H 4450 500 60  0000 C CNN
-F 2 "digital:Lattice_QFN48" H 4150 2000 60  0001 C CNN
-F 3 "https://www.mouser.com/ProductDetail/Lattice/ICE5LP1K-SG48ITR50?qs=sGAEpiMZZMvwLjDpJZyitJNdMN%2fKEQTHJMj%2fImmOWHhZL2XTDh5gKQ%3d%3d" H 4150 2000 60  0001 C CNN
-	1    4150 2000
-	1    0    0    -1
-$EndComp
-$Comp
-L ICE5LP1K-SG48ITR50 U301
 U 2 1 5AD190D4
 P 4800 4300
@@
 $EndComp
 $Comp
-L C_Small C303
-U 1 1 5AD222CE
-P 5100 2400
-F 0 "C303" H 5110 2470 50  0000 L CNN
-F 1 "10u" H 5110 2320 50  0000 L CNN
-F 2 "Capacitors_SMD:C_0805_HandSoldering" H 5100 2400 50  0001 C CNN
-F 3 "" H 5100 2400 50  0001 C CNN
-	1    5100 2400
-	1    0    0    -1
-$EndComp
-$Comp
-L GND #PWR078
-U 1 1 5AD22387
-P 5100 2600
-F 0 "#PWR078" H 5100 2350 50  0001 C CNN
-F 1 "GND" H 5100 2450 50  0000 C CNN
-F 2 "" H 5100 2600 50  0001 C CNN
-F 3 "" H 5100 2600 50  0001 C CNN
-	1    5100 2600
-	1    0    0    -1
-$EndComp
-$Comp
 L R_Small R307
 U 1 1 5AD22DF0
@@
 $EndComp
 $Comp
-L GND #PWR079
+L GND #PWR078
 U 1 1 5AD23697
 P 2850 5950
-F 0 "#PWR079" H 2850 5700 50  0001 C CNN
+F 0 "#PWR078" H 2850 5700 50  0001 C CNN
 F 1 "GND" H 2850 5800 50  0000 C CNN
 F 2 "" H 2850 5950 50  0001 C CNN
@@
 $EndComp
 $Comp
-L GND #PWR080
+L GND #PWR079
 U 1 1 5AD236F1
 P 3150 5950
-F 0 "#PWR080" H 3150 5700 50  0001 C CNN
+F 0 "#PWR079" H 3150 5700 50  0001 C CNN
 F 1 "GND" H 3150 5800 50  0000 C CNN
 F 2 "" H 3150 5950 50  0001 C CNN
@@
 	0    -1   -1   0
 $EndComp
-Text HLabel 6250 5500 0    60   Input ~ 0
+Text HLabel 3150 3800 0    60   Input ~ 0
 SPI0_CSN
-Text HLabel 6250 5200 0    60   Input ~ 0
+Text HLabel 3150 3500 0    60   Input ~ 0
 SPI0_MOSI
-Text HLabel 6250 5300 0    60   Input ~ 0
+Text HLabel 3150 3700 0    60   Input ~ 0
 SPI0_CLK
-Text HLabel 6250 5400 0    60   Input ~ 0
+Text HLabel 3150 3600 0    60   Input ~ 0
 SPI0_MISO
 $Comp
@@
 $EndComp
 $Comp
-L GND #PWR081
+L GND #PWR080
 U 1 1 5AD29C30
 P 3250 3250
-F 0 "#PWR081" H 3250 3000 50  0001 C CNN
+F 0 "#PWR080" H 3250 3000 50  0001 C CNN
 F 1 "GND" H 3250 3100 50  0000 C CNN
 F 2 "" H 3250 3250 50  0001 C CNN
@@
 $EndComp
 $Comp
-L GND #PWR082
+L GND #PWR081
 U 1 1 5AD2AF94
 P 3450 3250
-F 0 "#PWR082" H 3450 3000 50  0001 C CNN
+F 0 "#PWR081" H 3450 3000 50  0001 C CNN
 F 1 "GND" H 3450 3100 50  0000 C CNN
 F 2 "" H 3450 3250 50  0001 C CNN
@@
 Text HLabel 4100 4950 0    60   Input ~ 0
 SPI1_MOSI
-Text HLabel 4100 5050 0    60   Input ~ 0
+Text HLabel 4100 5150 0    60   Input ~ 0
 SPI1_MISO
-Text HLabel 4100 5150 0    60   Input ~ 0
-SPI1_SCK
 Text HLabel 4100 5250 0    60   Input ~ 0
 SPI1_CSN
-Text HLabel 5900 1550 0    60   Input ~ 0
+Text HLabel 5900 1850 0    60   Input ~ 0
 PLL_CLK
+Text HLabel 5900 1750 0    60   Input ~ 0
+PLL_DATA
 Text HLabel 5900 1650 0    60   Input ~ 0
-PLL_DATA
-Text HLabel 5900 1750 0    60   Input ~ 0
 PLL_LE
-Text HLabel 5900 1850 0    60   Input ~ 0
+Text HLabel 3400 2450 0    60   Input ~ 0
 PLL_MUXOUT
 Wire Wire Line
@@
 Wire Wire Line
 	6350 3000 6750 3000
-Wire Wire Line
-	5100 2250 6200 2250
 Wire Wire Line
 	6200 2250 6200 2700
@@
 	2400 3150 2300 3150
 Connection ~ 2400 2950
-Wire Wire Line
-	5100 2300 5100 2250
-Connection ~ 5350 2250
-Wire Wire Line
-	5100 2500 5100 2600
 Wire Wire Line
 	2100 4600 2100 4750
@@
 	6450 3200 6750 3200
 Wire Wire Line
-	6250 5500 6650 5500
-Wire Wire Line
-	6250 5400 6650 5400
-Wire Wire Line
-	6250 5300 6650 5300
-Wire Wire Line
-	6250 5200 6650 5200
-Wire Wire Line
 	4100 5250 4600 5250
 Wire Wire Line
@@
 Wire Wire Line
 	6400 1650 5900 1650
-Wire Wire Line
-	5900 1550 6450 1550
-Wire Wire Line
-	6450 1550 6450 2200
-Wire Wire Line
-	6450 2200 6750 2200
 Text Label 5900 3350 0    60   ~ 0
 CLK_40MHz
@@
 CLK_40MHz
 $Comp
-L GND #PWR083
+L GND #PWR082
 U 1 1 5AD30B62
 P 10100 3150
-F 0 "#PWR083" H 10100 2900 50  0001 C CNN
+F 0 "#PWR082" H 10100 2900 50  0001 C CNN
 F 1 "GND" H 10100 3000 50  0000 C CNN
 F 2 "" H 10100 3150 50  0001 C CNN
@@
 	10100 2950 9900 2950
 $Comp
-L +3V3 #PWR084
+L +3V3 #PWR083
 U 1 1 5AD30C79
 P 9100 2600
-F 0 "#PWR084" H 9100 2450 50  0001 C CNN
+F 0 "#PWR083" H 9100 2450 50  0001 C CNN
 F 1 "+3V3" H 9100 2740 50  0000 C CNN
 F 2 "" H 9100 2600 50  0001 C CNN
@@
 Connection ~ 9100 2750
 $Comp
-L GND #PWR085
+L GND #PWR084
 U 1 1 5AD30FF1
 P 9000 3150
-F 0 "#PWR085" H 9000 2900 50  0001 C CNN
+F 0 "#PWR084" H 9000 2900 50  0001 C CNN
 F 1 "GND" H 9000 3000 50  0000 C CNN
 F 2 "" H 9000 3150 50  0001 C CNN
@@
 Connection ~ 2850 5550
 $Comp
-L GND #PWR086
+L GND #PWR085
 U 1 1 5ADAED82
 P 2050 6000
-F 0 "#PWR086" H 2050 5750 50  0001 C CNN
+F 0 "#PWR085" H 2050 5750 50  0001 C CNN
 F 1 "GND" H 2050 5850 50  0000 C CNN
 F 2 "" H 2050 6000 50  0001 C CNN
@@
 	2050 5900 2050 6000
 $Comp
-L +3.3V #PWR087
+L +3.3V #PWR086
 U 1 1 5ADAF0F0
 P 1450 5450
-F 0 "#PWR087" H 1450 5300 50  0001 C CNN
+F 0 "#PWR086" H 1450 5300 50  0001 C CNN
 F 1 "+3.3V" H 1450 5590 50  0000 C CNN
 F 2 "" H 1450 5450 50  0001 C CNN
@@
 Connection ~ 1200 5550
 $Comp
-L GND #PWR088
+L GND #PWR087
 U 1 1 5ADAFCDD
 P 1200 5900
-F 0 "#PWR088" H 1200 5650 50  0001 C CNN
+F 0 "#PWR087" H 1200 5650 50  0001 C CNN
 F 1 "GND" H 1200 5750 50  0000 C CNN
 F 2 "" H 1200 5900 50  0001 C CNN
@@
 $EndComp
 $Comp
-L GND #PWR089
+L GND #PWR088
 U 1 1 5ADAFD55
 P 1050 5900
-F 0 "#PWR089" H 1050 5650 50  0001 C CNN
+F 0 "#PWR088" H 1050 5650 50  0001 C CNN
 F 1 "GND" H 1050 5750 50  0000 C CNN
 F 2 "" H 1050 5900 50  0001 C CNN
@@
 NoConn ~ 3950 2250
 NoConn ~ 3950 2350
-NoConn ~ 3950 2450
-NoConn ~ 3950 2950
-NoConn ~ 3950 3050
-NoConn ~ 3950 3150
-NoConn ~ 3950 3250
 NoConn ~ 6750 2800
 NoConn ~ 6750 2900
@@
 NoConn ~ 4600 5450
 NoConn ~ 4600 4450
+$Comp
+L TLV74312PDBVR U305
+U 1 1 5AD79ED3
+P 9200 4400
+F 0 "U305" H 9200 4550 60  0000 C CNN
+F 1 "TLV74312PDBVR" H 9550 4100 60  0000 C CNN
+F 2 "TO_SOT_Packages_SMD:SOT-23-5_HandSoldering" H 9200 4400 60  0001 C CNN
+F 3 "https://www.mouser.com/ProductDetail/Texas-Instruments/TLV74312PDBVR?qs=sGAEpiMZZMt1hubY80%2fs8Ncl2sHGlOOHyBzft4Bfjyk4ozWAIIKuIg%3d%3d" H 9200 4400 60  0001 C CNN
+	1    9200 4400
+	1    0    0    -1
+$EndComp
+$Comp
+L GND #PWR089
+U 1 1 5AD7A448
+P 9200 4850
+F 0 "#PWR089" H 9200 4600 50  0001 C CNN
+F 1 "GND" H 9200 4700 50  0000 C CNN
+F 2 "" H 9200 4850 50  0001 C CNN
+F 3 "" H 9200 4850 50  0001 C CNN
+	1    9200 4850
+	1    0    0    -1
+$EndComp
+Wire Wire Line
+	9200 4850 9200 4750
+$Comp
+L +3.3V #PWR090
+U 1 1 5AD7A575
+P 8750 4300
+F 0 "#PWR090" H 8750 4150 50  0001 C CNN
+F 1 "+3.3V" H 8750 4440 50  0000 C CNN
+F 2 "" H 8750 4300 50  0001 C CNN
+F 3 "" H 8750 4300 50  0001 C CNN
+	1    8750 4300
+	1    0    0    -1
+$EndComp
+Wire Wire Line
+	8750 4300 8750 4400
+Wire Wire Line
+	8300 4400 8850 4400
+$Comp
+L +1V2 #PWR091
+U 1 1 5AD7A6A3
+P 9650 4300
+F 0 "#PWR091" H 9650 4150 50  0001 C CNN
+F 1 "+1V2" H 9650 4440 50  0000 C CNN
+F 2 "" H 9650 4300 50  0001 C CNN
+F 3 "" H 9650 4300 50  0001 C CNN
+	1    9650 4300
+	1    0    0    -1
+$EndComp
+Wire Wire Line
+	9650 4300 9650 4400
+$Comp
+L C_Small C321
+U 1 1 5AD7B0F3
+P 8300 4600
+F 0 "C321" H 8310 4670 50  0000 L CNN
+F 1 "100n" H 8310 4520 50  0000 L CNN
+F 2 "Capacitors_SMD:C_0603_HandSoldering" H 8300 4600 50  0001 C CNN
+F 3 "" H 8300 4600 50  0001 C CNN
+	1    8300 4600
+	-1   0    0    -1
+$EndComp
+$Comp
+L C_Small C322
+U 1 1 5AD7B0F9
+P 8550 4600
+F 0 "C322" H 8560 4670 50  0000 L CNN
+F 1 "10u" H 8560 4520 50  0000 L CNN
+F 2 "Capacitors_SMD:C_0805_HandSoldering" H 8550 4600 50  0001 C CNN
+F 3 "" H 8550 4600 50  0001 C CNN
+	1    8550 4600
+	-1   0    0    -1
+$EndComp
+$Comp
+L GND #PWR092
+U 1 1 5AD7B0FF
+P 8300 4800
+F 0 "#PWR092" H 8300 4550 50  0001 C CNN
+F 1 "GND" H 8300 4650 50  0000 C CNN
+F 2 "" H 8300 4800 50  0001 C CNN
+F 3 "" H 8300 4800 50  0001 C CNN
+	1    8300 4800
+	-1   0    0    -1
+$EndComp
+$Comp
+L GND #PWR093
+U 1 1 5AD7B105
+P 8550 4800
+F 0 "#PWR093" H 8550 4550 50  0001 C CNN
+F 1 "GND" H 8550 4650 50  0000 C CNN
+F 2 "" H 8550 4800 50  0001 C CNN
+F 3 "" H 8550 4800 50  0001 C CNN
+	1    8550 4800
+	-1   0    0    -1
+$EndComp
+Wire Wire Line
+	8550 4700 8550 4800
+Wire Wire Line
+	8300 4700 8300 4800
+Wire Wire Line
+	8300 4400 8300 4500
+Wire Wire Line
+	8550 4400 8550 4500
+Connection ~ 8750 4400
+Connection ~ 8550 4400
+Wire Wire Line
+	8700 4400 8700 4550
+Wire Wire Line
+	8700 4550 8850 4550
+Connection ~ 8700 4400
+Wire Wire Line
+	9650 4400 9550 4400
+Wire Wire Line
+	5350 2250 6200 2250
+Text HLabel 4100 5050 0    60   Input ~ 0
+SPI1_SCK
+Wire Wire Line
+	3400 2450 3950 2450
+$Comp
+L ICE5LP1K-SG48ITR50 U301
+U 1 1 5AD1908F
+P 4150 2000
+F 0 "U301" H 4150 2000 60  0000 C CNN
+F 1 "ICE5LP1K-SG48ITR50" H 4450 500 60  0000 C CNN
+F 2 "digital:Lattice_QFN48" H 4150 2000 60  0001 C CNN
+F 3 "https://www.mouser.com/ProductDetail/Lattice/ICE5LP1K-SG48ITR50?qs=sGAEpiMZZMvwLjDpJZyitJNdMN%2fKEQTHJMj%2fImmOWHhZL2XTDh5gKQ%3d%3d" H 4150 2000 60  0001 C CNN
+	1    4150 2000
+	1    0    0    -1
+$EndComp
+Wire Wire Line
+	3950 2950 3550 2950
+Wire Wire Line
+	3550 2950 3550 3500
+Wire Wire Line
+	3550 3500 3150 3500
+Wire Wire Line
+	3150 3600 3600 3600
+Wire Wire Line
+	3600 3600 3600 3050
+Wire Wire Line
+	3600 3050 3950 3050
+Wire Wire Line
+	3950 3150 3650 3150
+Wire Wire Line
+	3650 3150 3650 3700
+Wire Wire Line
+	3650 3700 3150 3700
+Wire Wire Line
+	3150 3800 3700 3800
+Wire Wire Line
+	3700 3800 3700 3250
+Wire Wire Line
+	3700 3250 3950 3250
+NoConn ~ 3950 2650
+NoConn ~ 6650 5200
+NoConn ~ 6650 5300
+NoConn ~ 6650 5400
+NoConn ~ 6650 5500
 $EndSCHEMATC
