File: digital/digital.kicad_pcb (KiCad board)
At the start: 2 copper layers, 52 x 68 mm, 127 parts, among them J101 BASEBAND, J102 LNA_INTERFACE, J103 VCO_INTERFACE, J104 RF_POWER, J105 UART, J106 PLL_INTERFACE, J107 PA_INTERFACE, J108 USB_OTG, J109 FPGA_PROG, J110 SWD/JTAG, J111 PWR_IN, Q101 Q_PMOS_GSD, U101 LDK320AM33R, U102 TPS54308, U201 STM32F070C6T6, U202 SG5032CAN8.000000M-TJGA3, U301 ICE5LP1K-SG48ITR50, U302 LFSPXO025559Reel, U303 AT25SF041, U304 TLV74125PDBVR, U401 ADS7057, U402 LDK320AM33R, U403 OPA2376QDGKRQ1

Commit message: Finish digital layout
Parts:
- removed C303: 10u, Capacitors_SMD:C_0805_HandSoldering
- removed TP206: TEST, Connectors:PINTST
- added C321: 100n, Capacitors_SMD:C_0603_HandSoldering, F.Cu at (104.2, 121.2)
- added C322: 10u, Capacitors_SMD:C_0805_HandSoldering, F.Cu at (104.2, 122.8)
- added U305: TLV74312PDBVR, TO_SOT_Packages_SMD:SOT-23-5_HandSoldering, F.Cu at (104.3, 118.0)
- C203, C205, C206, C207, C208, C209, C210, C301, C302, C304, C305, C306, C307, C308, C309, C311, C312, C313, C314, C315, C316, C317, C318, C319, C320, D201, D401, D402, J110, J111, R101, R201, R302, R303, R401, R402, R404, R406, R407, R408, R409, R410, U304, U403: moved to F.Cu
- TP101, TP102, TP103, TP104, TP105, TP201: footprint Connectors:PINTST -> Measurement_Points:Measurement_Point_Round-SMD-Pad_Small
- TP202, TP203, TP204, TP205: footprint Connectors:PINTST -> Measurement_Points:Measurement_Point_Round-SMD-Pad_Small; moved to F.Cu
- moved RV401 191.4 mm to (106.4, 130.9), turned to 180 degrees
- moved U403 179.2 mm to (111.4, 145.0), turned to 180 degrees
- moved J105 172.7 mm to (146.7, 154.7), turned to 90 degrees
- moved R405 170.8 mm to (113.5, 149.6), turned to 180 degrees
- moved R406 170.5 mm to (117.6, 144.9), turned to 270 degrees
- moved R403 166.5 mm to (113.5, 147.8)
- moved R402 163.3 mm to (115.5, 148.4)
- moved U402 160.9 mm to (122.5, 140.2)
- moved U401 159.7 mm to (114.1, 133.8), turned to 90 degrees
- moved C104 159.5 mm to (124.9, 163.4), turned to 90 degrees
- moved C407 158.8 mm to (110.4, 144.9), turned to 90 degrees
- moved C408 158.4 mm to (112.2, 145.0), turned to 90 degrees
- moved R404 157.8 mm to (117.6, 148.4)
- moved C405 157.1 mm to (118.9, 133.7), turned to 90 degrees
- moved C406 156.9 mm to (116.8, 133.7), turned to 90 degrees
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Connections:
- J109 pad 2: /FLASH_SCK -> (no net)
- J109 pad 3: /FLASH_MISO -> /FLASH_CSN
- J109 pad 4: /FLASH_MOSI -> /FLASH_MISO
- J109 pad 5: /FLASH_CSN -> /FLASH_MOSI
- J109 pad 6: /FPGA_RSTN -> /FLASH_SCK
- J109 pad 7: (no net) -> /FPGA_RSTN
- U201 pad 13: (no net) -> /PA_EN
- U201 pad 2: (no net) -> /LNA2_EN
- U201 pad 26: /PA_EN -> (no net)
- U201 pad 27: /LNA1_EN -> (no net)
- U201 pad 28: /LNA2_EN -> (no net)
- U201 pad 3: (no net) -> /LNA1_EN
- U301 pad 10: (no net) -> /FPGA/SPI0_MISO
- U301 pad 11: (no net) -> /FPGA/SPI0_CLK
- U301 pad 12: (no net) -> /FPGA/SPI0_CSN
- U301 pad 19: /ADC/ADC_MISO -> /ADC/ADC_SCK
- U301 pad 20: /ADC/ADC_SCK -> /ADC/ADC_MISO
- U301 pad 25: /PLL_CLK -> (no net)
- U301 pad 26: /PLL_DATA -> /PLL_LE
- U301 pad 27: /PLL_LE -> /PLL_DATA
- U301 pad 28: /PLL_MUXOUT -> /PLL_CLK
- U301 pad 4: (no net) -> /PLL_MUXOUT
- U301 pad 45: /FPGA/SPI0_MOSI -> (no net)
- U301 pad 46: /FPGA/SPI0_CLK -> (no net)
- U301 pad 47: /FPGA/SPI0_MISO -> (no net)
- U301 pad 48: /FPGA/SPI0_CSN -> (no net)
- U301 pad 9: (no net) -> /FPGA/SPI0_MOSI
Routing:
- net GND: track 0.00 -> 553.3 mm, vias 0 -> 34
- net +3V3: track 0.00 -> 319.5 mm, vias 0 -> 21
- net +5V: track 0.00 -> 112.1 mm, vias 0 -> 4
- net +1V2: track 0.00 -> 49.1 mm, vias 0 -> 2
- net /STM32_RSTN: track 0.00 -> 38.5 mm, vias 0 -> 7
- net Net-(C405-Pad1): track 0.00 -> 32.2 mm, vias 0 -> 3
- net /FPGA/SPI0_MISO: track 0.00 -> 31.5 mm, vias 0 -> 1
- net /FLASH_MISO: track 0.00 -> 31.4 mm, vias 0 -> 1
- net /FLASH_SCK: track 0.00 -> 30.5 mm, vias 0 -> 1
- net /UART_RX: track 0.00 -> 30.0 mm, vias 0 -> 1
- net /LNA1_EN: track 0.00 -> 29.9 mm
- net /FPGA/CDONE: track 0.00 -> 29.6 mm
- net /ADC/ADC_MISO: track 0.00 -> 29.3 mm, vias 0 -> 2
- net /FPGA/SPI0_CLK: track 0.00 -> 29.0 mm, vias 0 -> 1
- net /ADC/ADC_CSN: track 0.00 -> 28.2 mm
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- added copper zone on B.Cu, net GND
- added copper zone on F.Cu, net GND
Other:
- net class Default: clearance 0.2 -> 0.1524; trace_width 0.25 -> 0.1524; via_dia 0.6 -> 0.6858; via_drill 0.4 -> 0.3302
- rule trace_clearance: 0.2 -> 0.1524
- rule trace_min: 0.2 -> 0.1524
- rule via_min_drill: 0.3 -> 0.3302
- rule via_min_size: 0.4 -> 0.6858

Commit message: Fix up some minor things
Routing:
- net GND: track 553.3 -> 564.8 mm, vias 34 -> 35
- net +5V: track 112.1 -> 109.1 mm
- net /STM32_BOOT: track 23.0 -> 24.2 mm, vias 0 -> 2
- net +3V3: track 319.5 -> 320.3 mm

Commit message: Regenerate Gerbers
Parts:
- added J101: BASEBAND, Pin_Headers:Pin_Header_Straight_1x02_Pitch2.54mm, F.Cu at (110.0, 153.5)
Changed lines of the file:
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@@
     (links 284)
     (no_connects 0)
-    (area 91.5 95.25 156.950001 174.900001)
+    (area 99.924999 99.924999 152.075001 168.075001)
     (thickness 1.6)
     (drawings 4)
     (tracks 1202)
     (zones 0)
-    (modules 128)
+    (modules 129)
     (nets 71)
   )
@@
   )
   (setup
-    (last_trace_width 0.8)
+    (last_trace_width 0.1524)
     (user_trace_width 0.3)
     (user_trace_width 0.4)
@@
     (visible_elements FFFFFF7F)
     (pcbplotparams
-      (layerselection 0x00030_80000001)
+      (layerselection 0x01030_80000001)
       (usegerberextensions false)
       (excludeedgelayer true)
@@
       (outputformat 1)
       (mirror false)
-      (drillshape 1)
+      (drillshape 0)
       (scaleselection 1)
-      (outputdirectory ""))
+      (outputdirectory ../gerber/))
   )
   (net 0 "")
@@
     (add_net VBUS)
   )
+  (module Pin_Headers:Pin_Header_Straight_1x02_Pitch2.54mm (layer F.Cu)
+    (at 110.05 153.46)
+    (descr "Through hole straight pin header, 1x02, 2.54mm pitch, single row")
+    (tags "Through hole pin header THT 1x02 2.54mm single row")
+    (fp_text reference J101 (at 0 -2.33) (layer F.SilkS)
+      (effects (font (size 1 1) (thickness 0.15)))
+    )
+    (fp_text value BASEBAND (at 0 4.87) (layer F.Fab)
+      (effects (font (size 1 1) (thickness 0.15)))
+    )
+    (fp_line (start -0.635 -1.27) (end 1.27 -1.27) (layer F.Fab) (width 0.1))
+    (fp_line (start 1.27 -1.27) (end 1.27 3.81) (layer F.Fab) (width 0.1))
+    (fp_line (start 1.27 3.81) (end -1.27 3.81) (layer F.Fab) (width 0.1))
+    (fp_line (start -1.27 3.81) (end -1.27 -0.635) (layer F.Fab) (width 0.1))
+    (fp_line (start -1.27 -0.635) (end -0.635 -1.27) (layer F.Fab) (width 0.1))
+    (fp_line (start -1.33 3.87) (end 1.33 3.87) (layer F.SilkS) (width 0.12))
+    (fp_line (start -1.33 1.27) (end -1.33 3.87) (layer F.SilkS) (width 0.12))
+    (fp_line (start 1.33 1.27) (end 1.33 3.87) (layer F.SilkS) (width 0.12))
+    (fp_line (start -1.33 1.27) (end 1.33 1.27) (layer F.SilkS) (width 0.12))
+    (fp_line (start -1.33 0) (end -1.33 -1.33) (layer F.SilkS) (width 0.12))
+    (fp_line (start -1.33 -1.33) (end 0 -1.33) (layer F.SilkS) (width 0.12))
+    (fp_line (start -1.8 -1.8) (end -1.8 4.35) (layer F.CrtYd) (width 0.05))
+    (fp_line (start -1.8 4.35) (end 1.8 4.35) (layer F.CrtYd) (width 0.05))
+    (fp_line (start 1.8 4.35) (end 1.8 -1.8) (layer F.CrtYd) (width 0.05))
+    (fp_line (start 1.8 -1.8) (end -1.8 -1.8) (layer F.CrtYd) (width 0.05))
+    (fp_text user %R (at 0 1.27 90) (layer F.Fab)
+      (effects (font (size 1 1) (thickness 0.15)))
+    )
+    (pad 1 thru_hole rect (at 0 0) (size 1.7 1.7) (drill 1) (layers *.Cu *.Mask)
+      (net 28 /ADC/IN+))
+    (pad 2 thru_hole oval (at 0 2.54) (size 1.7 1.7) (drill 1) (layers *.Cu *.Mask)
+      (net 29 /ADC/IN-))
+    (model ${KISYS3DMOD}/Pin_Headers.3dshapes/Pin_Header_Straight_1x02_Pitch2.54mm.wrl
+      (at (xyz 0 0 0))
+      (scale (xyz 1 1 1))
+      (rotate (xyz 0 0 0))
+    )
+  )
   (module Capacitors_SMD:C_0805_HandSoldering (layer B.Cu)
